File: Schematics & PCB/Owen's Learning Environment (bad)/_autosave-salp_board.kicad_sch (KiCad schematic)
At the start: 31 parts, among them U1 ATtiny3226-S, U2 PN5321A3HN/C106_55, U3 BMI270, Y1 27.12 MHz

Commit message: Significant Overhaul
- was a bit too much work to write my own libraries, so implemented a few for now (with licenses) for now. will have to be optimized since the current memory usage is insanely high [3031/3072, 98.7% RAM] and [17597/32768, 53.7% Flash]
Parts:
- removed C1, C2: 200p, symbol Device:C
- removed C10, C14, C16, C7, C8: .1u, symbol Device:C
- removed C11: 1n, symbol Device:C
- removed C12, C13: 22pF, symbol Device:C
- removed C15: 10uF, symbol Device:C
- removed C3, C4: 22p, symbol Device:C
- removed C5, C6: 220p, symbol Device:C
- removed C9: 4.7u, symbol Device:C
- removed L1, L2: 560nH, symbol Device:L
- removed R1: 1.6K, symbol Device:R_Small_US
- removed R2: 1K, symbol Device:R_Small_US
- removed R3, R4: 4.7k, Resistor_SMD:R_0402_1005Metric_Pad0.72x0.64mm_HandSolder, symbol Device:R_Small_US
- removed R5, R7, R8: 10k, symbol Device:R_Small_US
- removed R6: 20k, symbol Device:R_Small_US
- removed R9: 10K, Resistor_SMD:R_0402_1005Metric_Pad0.72x0.64mm_HandSolder, symbol Device:R_Small_US
- removed U1: ATtiny3226-S, Package_SO:SOIC-20W_7.5x12.8mm_P1.27mm, symbol MCU_Microchip_ATtiny:ATtiny3226-S
- removed U2: PN5321A3HN/C106_55, HVQFN40_SOT618-1_NXP, symbol Orb_library:PN5321A3HN_C106_55
- removed U3: BMI270, BMI270_BOS, symbol salp:BMI270
- removed Y1: 27.12 MHz, symbol Device:Crystal
Connections:
- no-connect marks 17 -> 0
Other:
- added sheet PN532 (PN532.sch.kicad_sch)
- note removed: "IRQ: See 2.4.2.1 Application Note"
- note removed: "P37-29 are unusued: SPI/HSU See Application Note"
