File: Schematics & PCB/Owen's Learning Environment (bad)/_autosave-salp_board.kicad_sch (KiCad schematic)
At the start: 43 parts, among them J1 ATTINY3226, J10 POWER, J11 UPDI, J2 Conn_01x01, J3 Conn_01x01, J4 Conn_Coaxial_Small, J5 Conn_Coaxial_Small, J6 Conn_01x01, J7 Conn_Coaxial_Small, J8 ATTINY3226, J9 POWER_JUMPER, SW1 SW_DIP_x02, U1 LD1117S33TR, U2 PN5321A3HN/C106_55, U3 ATtiny3226-S, Y1 27.12 MHz

Commit message: Added some stuff to the PN532
- buffer reading and checking (need to change)
Parts:
- removed J11: UPDI, Connector_PinSocket_2.54mm:PinSocket_1x03_P2.54mm_Vertical, symbol Connector_Generic:Conn_01x03
- added J12: ~, Connector_PinHeader_2.54mm:PinHeader_1x06_P2.54mm_Horizontal, symbol Connector_Generic:Conn_01x06
Connections:
- net AVDD: no longer C14.1, C15.1, C7.1, C9.1, SW1.1, SW1.2, U2.39 (DVDD), U2.5 (TVDD)
- net GND: now also J12.6 (Pin_6)
- net PB2: now also J12.2 (Pin_2)
- net PB3: now also J12.3 (Pin_3)
- net V_USB: now also J12.4 (Pin_4)
- new net DVDD: C14.1, C15.1, SW1.1, SW1.2, U2.39 (DVDD)
- new net TVDD: C7.1, C9.1, U2.5 (TVDD)
- no-connect marks 12 -> 14
Other:
- note added: "Serial/FTDI Header"
- moved on the sheet: C21, C22, C23, U1
