File: Schematics & PCB/Owen's Learning Environment (bad)/salp_board.kicad_sch (KiCad schematic)
At the start: 37 parts, among them J1 ATTINY3226, J10 POWER, J2 Conn_01x01, J3 Conn_01x01, J4 Conn_Coaxial_Small, J5 Conn_Coaxial_Small, J6 Conn_01x01, J7 Conn_Coaxial_Small, J8 ATTINY3226, J9 POWER_JUMPER, U2 PN5321A3HN/C106_55, U3 ATtiny3226-S, Y1 27.12 MHz

Commit message: Added some stuff to the PN532
- buffer reading and checking (need to change)
Parts:
- added C21, C23: 100nF, Capacitor_SMD:C_0805_2012Metric_Pad1.18x1.45mm_HandSolder, symbol Device:C
- added C22: 10uF, Capacitor_SMD:C_0805_2012Metric_Pad1.18x1.45mm_HandSolder, symbol Device:C
- added J11: UPDI, Connector_PinSocket_2.54mm:PinSocket_1x03_P2.54mm_Vertical, symbol Connector_Generic:Conn_01x03
- added J12: ~, Connector_PinHeader_2.54mm:PinHeader_1x06_P2.54mm_Horizontal, symbol Connector_Generic:Conn_01x06
- added SW1: SW_DIP_x02, symbol Switch:SW_DIP_x02
- added U1: LD1117S33TR, Package_TO_SOT_SMD:SOT-223-3_TabPin2, symbol Regulator_Linear:LD1117S33TR_SOT223
- C14, C8: value .1u -> 100 nF
Connections:
- net I1 is gone; now on net GND: U2.17 (I1)
- net IO is gone; now on net GND: U2.16 (I0)
- net PVDD is gone; now on net PA7: U2.38 (RSTPD_N)
- net +3.3V: now also C23.1, J11.1 (Pin_1); no longer C14.1, C15.1, C7.1, C8.1, C9.1, U2.39 (DVDD), U2.5 (TVDD)
- net AVDD: now also C8.1
- net GND: now also C21.2, C22.2, C23.2, J11.2 (Pin_2), J12.6 (Pin_6), SW1.3, SW1.4, U1.1 (GND)
- net PA0: now also J11.3 (Pin_3)
- net PB2: now also J12.2 (Pin_2)
- net PB3: now also J12.3 (Pin_3)
- net VCC: now also C21.1, U1.3 (VI)
- net V_REG: now also C22.1, U1.2 (VO)
- net V_USB: now also J12.4 (Pin_4)
- new net DVDD: C14.1, C15.1, SW1.1, SW1.2, U2.39 (DVDD)
- new net TVDD: C7.1, C9.1, U2.5 (TVDD)
- no-connect marks 12 -> 14
Other:
- note added: "Decoupling (DVDD, AVDD, TVDD) DVDD and TVDD made based on PN532_C1 s13"
- note added: "I/O Toggle Should be set to I2C by default (IO -> DVDD, I1 -> GND)"
- note added: "OSCILLATOR See User Manual 8.5.2"
- note added: "PA7: RSTPD_N for PN532"
- note added: "RF SECTION: See AN1445 Antenna Design Guide EMC Filter: TX1-TX2, L1, L2, C5, C6 Reduces harmonics and performs impedance transformation Matching Circuit: C1, C2, C3, C4 Acts as an impedance transformation block"
- note added: "Serial/FTDI Header"
- note added: "UPDI Header"
- note added: "VRM"
- moved on the sheet: C12, C13, C14, C15, C17, C7, C8, C9, U2, Y1
