File: Schematics & PCB/sensOrb/_autosave-salp_board.kicad_sch (KiCad schematic)
At the start: 59 parts, among them J1 ATTINY3226, J10 POWER, J4 Conn_01x03, J8 ATTINY3226, J9 POWER_JUMPER, Q1 IRLML6402, Q2 IRLML6402, SW1 SW_DIP_x02, SW2 SW_DPDT_x2, U1 LD1117S33TR, U2 PN5321A3HN/C106_55, U3 ATtiny3226-S, U4 TP4057, U6 DW01A, Y1 27.12 MHz

Commit message: Layout 1: No ERC/DRC done yet
Parts:
- J4: footprint (none) -> Connector_PinHeader_2.54mm:PinHeader_1x03_P2.54mm_Horizontal
Changed lines of the file:
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@@
 			)
 		)
-		(property "Footprint" ""
+		(property "Footprint" "Connector_PinHeader_2.54mm:PinHeader_1x03_P2.54mm_Horizontal"
 			(at 29.21 138.43 0)
 			(effects
