File: Schematics & PCB/sensOrb/salp_board.kicad_pcb (KiCad board)
At the start: 4 copper layers, 64.8 x 58.7 mm, 77 parts, among them J1 ATTINY3226, J10 POWER, J4 Conn_01x03, J8 ATTINY3226, J9 POWER_JUMPER, Q1 IRLML6402, Q2 IRLML6402, SW2 SW_DPDT_x2, U1 LD1117S33TR, U2 PN5321A3HN/C106_55, U3 ATtiny3226-S, U4 TP4057, U6 DW01A, Y2 27.12 MHz

Commit message: Flipped Battery Slot, Minor Edits
Parts:
- BT1: moved to B.Cu
Routing:
- net +BAT: track 72.3 -> 79.3 mm
- net Net-(J4-Pin_1): track 29.9 -> 35.3 mm
- net GND: track 109.8 -> 111.8 mm, vias 17 -> 16

Commit message: Fixes To SCH, 4-Layer PCB In Progress
Parts:
- added GND1: TestPoint, TestPoint:TestPoint_Pad_D1.0mm, F.Cu at (260.0, 49.5)
- H1, H2, H3, H4: value MountingHole -> MountingHole_Pad; footprint MountingHole:MountingHole_2.2mm_M2 -> MountingHole:MountingHole_2.2mm_M2_Pad
- moved C9 112.8 mm to (270.5, 78.5)
- moved C7 105.3 mm to (262.0, 74.5)
- moved I1 105.0 mm to (260.0, 38.5)
- moved R10 104.1 mm to (259.5, 96.5)
- moved C22 103.8 mm to (250.5, 85.0)
- moved C13 102.9 mm to (265.5, 78.5)
- moved PA3/SCK/P72 98.5 mm to (273.0, 44.5)
- moved C5 98.2 mm to (280.5, 85.5)
- moved C8 97.7 mm to (254.5, 75.5)
- moved C6 96.2 mm to (278.5, 81.5)
- moved C21 95.6 mm to (254.5, 85.0)
- moved C12 93.6 mm to (260.5, 79.0)
- moved I0 92.7 mm to (249.5, 44.5)
- moved TX2 92.3 mm to (257.0, 44.5)
- moved RX1 91.0 mm to (252.5, 38.5)
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Connections:
- C16 pad 1: VCC -> +3.3V
- C18 pad 1: VCC -> +3.3V
- C19 pad 1: VCC -> +3.3V
- U2 pad 23: VCC -> +3.3V
- U3 pad 1: VCC -> +3.3V
Routing:
- net +3.3V: track 101.6 -> 8.76 mm, vias 7 -> 6
- net VCC: track 80.6 -> 0.00 mm, vias 2 -> 0
- net GND: track 111.8 -> 54.1 mm, vias 16 -> 11
- net +BAT: track 79.3 -> 24.1 mm, vias 4 -> 1
- net /PA1: track 45.4 -> 8.13 mm
- net /PA7: track 42.6 -> 8.21 mm, vias 4 -> 0
- net /PA2: track 42.5 -> 9.22 mm
- net /PA3: track 41.4 -> 10.6 mm
- net Net-(J4-Pin_1): track 35.3 -> 5.08 mm
- net /V_USB: track 37.8 -> 60.2 mm
- net /PA4: track 30.6 -> 10.7 mm
- net /PA5: track 27.8 -> 9.26 mm, vias 3 -> 0
- net Net-(C4-Pad2): track 17.7 -> 0.00 mm
- net /V_REG: track 30.5 -> 15.2 mm, vias 2 -> 0
- net /OSCIN: track 15.0 -> 0.00 mm
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- added copper zone on In1.Cu, net +3.3V
- added copper zone on In2.Cu, net GND
- removed copper zone on B.Cu, net GND

Commit message: Updated Sch, Traces Routed, Needs Verification
Parts:
- removed R3: 4.7k, Resistor_SMD:R_0805_2012Metric_Pad1.20x1.40mm_HandSolder
- removed SW2: SW_DPDT_x2, Button_Switch_THT:SW_CK_JS202011CQN_DPDT_Straight
- added J2: READ/WRITE, Connector_PinHeader_2.54mm:PinHeader_1x03_P2.54mm_Vertical, F.Cu at (180.4, 102.0)
- added J3: READ/WRITE, Connector_PinHeader_2.54mm:PinHeader_1x03_P2.54mm_Vertical, F.Cu at (180.4, 106.0)
- moved C2 134.2 mm to (141.0, 71.5)
- moved C5 130.8 mm to (151.0, 67.0), turned to -90 degrees
- moved C1 129.3 mm to (141.0, 67.0)
- moved C6 127.9 mm to (151.0, 71.5), turned to -90 degrees
- moved C13 124.5 mm to (141.0, 81.0), turned to -90 degrees
- moved C4 123.5 mm to (146.0, 72.5), turned to 0 degrees
- moved C3 119.2 mm to (146.0, 66.0), turned to 0 degrees
- moved C12 109.5 mm to (151.0, 76.5), turned to 90 degrees
- moved C9 107.9 mm to (163.5, 64.5)
- moved C10 101.5 mm to (158.0, 76.0), turned to -90 degrees
- moved R1 100.4 mm to (155.5, 72.5), turned to 0 degrees
- moved C7 98.7 mm to (163.5, 67.0)
- moved C22 96.6 mm to (154.5, 96.0), turned to 90 degrees
- moved C11 93.5 mm to (161.5, 76.0), turned to -90 degrees
- moved L2 91.9 mm to (163.5, 69.5), turned to 0 degrees
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Connections:
- C14 pad 1: +3.3V -> /DVDD
- C15 pad 1: +3.3V -> /DVDD
- C7 pad 1: +3.3V -> /TVDD
- C8 pad 1: +3.3V -> /AVDD
- C9 pad 1: +3.3V -> /TVDD
- DVDD1 pad 1: +3.3V -> /DVDD
- I1 pad 1: +3.3V -> /DVDD
- U2 pad 17: +3.3V -> /DVDD
- U2 pad 39: +3.3V -> /DVDD
- U2 pad 5: +3.3V -> /TVDD
- U2 pad 8: +3.3V -> /AVDD
Routing:
- net +BAT: track 24.1 -> 94.1 mm, vias 1 -> 3
- net Net-(J4-Pin_1): track 5.08 -> 52.5 mm
- net VCC: track 0.00 -> 40.0 mm, vias 0 -> 1
- net GND: track 54.1 -> 93.3 mm, vias 11 -> 24
- net /OSCOUT: track 0.00 -> 34.3 mm
- net /PA1: track 8.13 -> 37.0 mm
- net /OSCIN: track 0.00 -> 26.5 mm
- net /PA2: track 9.22 -> 35.7 mm, vias 0 -> 3
- net /PA3: track 10.6 -> 34.9 mm
- net Net-(C3-Pad2): track 0.00 -> 23.0 mm
- net /PA7: track 8.21 -> 30.5 mm, vias 0 -> 1
- net /PA5: track 9.26 -> 30.4 mm, vias 0 -> 1
- net /DVDD: track 0.00 -> 20.4 mm, vias 0 -> 2
- net Net-(SW2B-C): track 18.9 -> 0.00 mm
- net Net-(C4-Pad2): track 0.00 -> 16.7 mm
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Other:
- board text removed: "Owen Pyle SIMlab 05/01/2025"
