File: Schematics & PCB/sensOrb/salp_board.kicad_pcb (KiCad board)
At the start: 4 copper layers, 64.8 x 58.7 mm, 78 parts, among them J1 ATTINY3226, J10 POWER, J2 READ/WRITE, J3 READ/WRITE, J4 Conn_01x03, J8 ATTINY3226, J9 POWER_JUMPER, Q1 IRLML6402, Q2 IRLML6402, U1 LD1117S33TR, U2 PN5321A3HN/C106_55, U3 ATtiny3226-S, U4 TP4057, U6 DW01A, Y2 27.12 MHz

Commit message: Fixes
Parts:
- removed +BAT1, DVDD1, GND1, I0, I1, PA1/MOSI/SDA/HSU_TX1, PA2/MISO/P71, PA3/SCK/P72, PA4/NSS/SCL/HSU_RX1, PA5/RSTPD_N1, PA7/IRQ1, PC1, PC2, PC3, RX1, TX1, TX2: TestPoint, TestPoint:TestPoint_Pad_D1.0mm
Routing:
- net Net-(U2-I0): track 0.00 -> 9.80 mm, vias 0 -> 2
- net Net-(J4-Pin_1): track 52.5 -> 57.6 mm
Other:
- board text added: "Initial Design by Owen Pyle Revisions by Jack Cunningham 6/23/25"

Commit message: Updated Silkscreen Again
Other:
- board text added: "PA0"
- board text added: "PA1"
- board text added: "PA2"
- board text added: "PA3"
- board text added: "PA4"
- board text added: "PA5"
- board text added: "PA6"
- board text added: "PA7"
- board text added: "PB2"
- board text added: "PB3"
- board text added: "PB4"
- board text added: "PB5"
- board text added: "PC0"
- board text added: "PC1"
- board text added: "PC2"
- board text added: "PC3"
- board text added: "SCL"
- board text added: "SDA"
Changed lines of the file:
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@@
+		)
+	)
+	(gr_text "PC0"
+		(at 195 100.5 0)
+		(layer "F.SilkS")
+		(effects
+			(font
+				(size 0.7 0.7)
+				(thickness 0.1)
+			)
+			(justify left bottom)
+		)
+	)
+	(gr_text "PB3"
+		(at 165.5 98 0)
+		(layer "F.SilkS")
+		(effects
+			(font
+				(size 0.5 0.5)
+				(thickness 0.1)
+			)
+			(justify left bottom)
+		)
+	)
+	(gr_text "PC3"
+		(at 195 93 0)
+		(layer "F.SilkS")
+		(effects
+			(font
+				(size 0.7 0.7)
+				(thickness 0.1)
+			)
+			(justify left bottom)
+		)
+	)
+	(gr_text "PA4"
+		(at 165.5 83 0)
+		(layer "F.SilkS")
+		(effects
+			(font
+				(size 0.5 0.5)
+				(thickness 0.1)
+			)
+			(justify left bottom)
 		)
 	)
@@
 		)
 	)
+	(gr_text "PA5\n"
+		(at 165.5 85 0)
+		(layer "F.SilkS")
+		(effects
+			(font
+				(size 0.5 0.5)
+				(thickness 0.1)
+			)
+			(justify left bottom)
+		)
+	)
+	(gr_text "PB5"
+		(at 165.5 92.5 0)
+		(layer "F.SilkS")
+		(effects
+			(font
+				(size 0.5 0.5)
+				(thickness 0.1)
+			)
+			(justify left bottom)
+		)
+	)
+	(gr_text "PA2"
+		(at 195 85.5 0)
+		(layer "F.SilkS")
+		(effects
+			(font
+				(size 0.7 0.7)
+				(thickness 0.1)
+			)
+			(justify left bottom)
+		)
+	)
+	(gr_text "PA0"
+		(at 195 90.5 0)
+		(layer "F.SilkS")
+		(effects
+			(font
+				(size 0.7 0.7)
+				(thickness 0.1)
+			)
+			(justify left bottom)
+		)
+	)
+	(gr_text "SCL"
+		(at 195 103 0)
+		(layer "F.SilkS")
+		(effects
+			(font
+				(size 0.7 0.7)
+				(thickness 0.1)
+			)
+			(justify left bottom)
+		)
+	)
+	(gr_text "PA1"
+		(at 195 88 0)
+		(layer "F.SilkS")
+		(effects
+			(font
+				(size 0.7 0.7)
+				(thickness 0.1)
+			)
+			(justify left bottom)
+		)
+	)
+	(gr_text "PC1"
+		(at 195 98 0)
+		(layer "F.SilkS")
+		(effects
+			(font
+				(size 0.7 0.7)
+				(thickness 0.1)
+			)
+			(justify left bottom)
+		)
+	)
+	(gr_text "PA3"
+		(at 195 83 0)
+		(layer "F.SilkS")
+		(effects
+			(font
+				(size 0.7 0.7)
+				(thickness 0.1)
+			)
+			(justify left bottom)
+		)
+	)
+	(gr_text "PA6"
+		(at 165.5 87.5 0)
+		(layer "F.SilkS")
+		(effects
+			(font
+				(size 0.5 0.5)
+				(thickness 0.1)
+			)
+			(justify left bottom)
+		)
+	)
+	(gr_text "PB2"
+		(at 165.5 100 0)
+		(layer "F.SilkS")
+		(effects
+			(font
+				(size 0.5 0.5)
+				(thickness 0.1)
+			)
+			(justify left bottom)
+		)
+	)
 	(gr_text "LEFT-Monitor\nRIGHT-Program"
 		(at 182.88512 114.344463 0)
@@
 			)
 			(justify left bottom)
+		)
+	)
+	(gr_text "PC2"
+		(at 195 95.5 0)
+		(layer "F.SilkS")
+		(effects
+			(font
+				(size 0.7 0.7)
+				(thickness 0.1)
+			)
+			(justify left bottom)
+		)
+	)
+	(gr_text "PB4\n"
+		(at 165.5 95.5 0)
+		(layer "F.SilkS")
+		(effects
+			(font
+				(size 0.5 0.5)
+				(thickness 0.1)
+			)
+			(justify left bottom)
+		)
+	)
+	(gr_text "SDA"
+		(at 165.5 103 0)
+		(layer "F.SilkS")
+		(effects
+			(font
+				(size 0.5 0.5)
+				(thickness 0.1)
+			)
+			(justify left bottom)
+		)
+	)
+	(gr_text "PA7"
+		(at 165.5 90 0)
+		(layer "F.SilkS")
+		(effects
+			(font
+				(size 0.5 0.5)
+				(thickness 0.1)
+			)
+			(justify left bottom)

Commit message: Updated Tracewidths
Parts:
- moved R6 1.00 mm to (153.5, 108.0)
Routing:
- net VCC: track 40.0 -> 78.6 mm
- net +BAT: track 94.1 -> 95.5 mm
- net /PC1: track 46.5 -> 47.7 mm
- net Net-(D5-B): track 10.1 -> 9.10 mm
- net /PB3: track 22.8 -> 22.3 mm

Commit message: Antenna Fix + DRC Fixes
Parts:
- moved J4 0.13 mm to (136.4, 71.5)
- turned C1 to -90 degrees
- turned C2 to -90 degrees
Connections:
- C1 pad 1: Net-(J4-Pin_1) -> Net-(J4-Pin_3)
- C1 pad 2: Net-(J4-Pin_1) -> Net-(J4-Pin_2)
- C2 pad 1: Net-(J4-Pin_1) -> Net-(J4-Pin_2)
- C3 pad 1: Net-(J4-Pin_1) -> Net-(J4-Pin_3)
- C5 pad 2: Net-(J4-Pin_1) -> Net-(J4-Pin_2)
- C6 pad 1: Net-(J4-Pin_1) -> Net-(J4-Pin_2)
- J4 pad 2: Net-(J4-Pin_1) -> Net-(J4-Pin_2)
- J4 pad 3: Net-(J4-Pin_1) -> Net-(J4-Pin_3)
Routing:
- net Net-(J4-Pin_1): track 57.6 -> 9.04 mm
- net Net-(J4-Pin_2): track 0.00 -> 20.2 mm
- net Net-(J4-Pin_3): track 0.00 -> 8.83 mm

Commit message: Tracewidth Fixes
Routing:
- net +BAT: track 95.5 -> 96.5 mm
- net /PA7: track 30.5 -> 31.2 mm
- net /PA2: vias 3 -> 1
