File: Schematics & PCB/sensOrb/salp_board.kicad_sch (KiCad schematic)
At the start: 59 parts, among them J1 ATTINY3226, J10 POWER, J4 Conn_01x03, J8 ATTINY3226, J9 POWER_JUMPER, Q1 IRLML6402, Q2 IRLML6402, SW1 SW_DIP_x02, SW2 SW_DPDT_x2, U1 LD1117S33TR, U2 PN5321A3HN/C106_55, U3 ATtiny3226-S, U4 TP4057, U6 DW01A, Y1 27.12 MHz

Commit message: Semi-finalized PCB design
Parts:
- removed R12: 1k, Resistor_SMD:R_0805_2012Metric_Pad1.20x1.40mm_HandSolder, symbol Device:R_Small_US
- removed SW1: SW_DIP_x02, Button_Switch_SMD:SW_DIP_SPSTx02_Slide_6.7x6.64mm_W8.61mm_P2.54mm_LowProfile, symbol Switch:SW_DIP_x02
- removed Y1: 27.12 MHz, Crystal:Crystal_SMD_3225-4Pin_3.2x2.5mm, symbol Device:Crystal
- added H1, H2, H3, H4: MountingHole, MountingHole:MountingHole_2.2mm_M2, symbol Mechanical:MountingHole
- added J2, J3: Conn_02x20_Counter_Clockwise, symbol Connector_Generic:Conn_02x20_Counter_Clockwise
- added Y2: 27.12 MHz, Crystal:Crystal_SMD_SeikoEpson_TSX3225-4Pin_3.2x2.5mm_HandSoldering, symbol Device:Crystal_GND24
- BT1: footprint Battery:Battery_Panasonic_CR2032-HFN_Horizontal_CircularHoles -> Battery:BatteryHolder_Keystone_1060_1x2032
- J4: footprint (none) -> Connector_PinHeader_2.54mm:PinHeader_1x03_P2.54mm_Horizontal
Connections:
- net IO is gone; now on an unnamed net: U2.16 (I0)
- net +3.3V: now also Q2.3 (D), U2.17 (I1)
- net GND: now also Y2.2, Y2.4; no longer D4.3, J9.1 (Pin_1)
- net OSCIN: now also Y2.1
- net OSCOUT: now also Y2.3
- net VCC: no longer Q2.3 (D)
- net I1: no longer names the net of R10.2
- net I1: no longer U2.17 (I1)
- new net VOR: D4.3, J9.1 (Pin_1)
Other:
- note added: "Mounting Holes"
- note removed: "I/O Toggle Should be set to SPI by default (IO -> GND, I1 -> DVDD)"
- moved on the sheet: BT1, C17, C21, C22, C23, D2, D3, D4, Q1, Q2, R10, R11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

Commit message: Board V1 - sent to fab (?)
Parts:
- added +BAT1, DVDD1, GND1, I0, I1, PA1/MOSI/SDA/HSU_TX1, PA2/MISO/P71, PA3/SCK/P72, PA4/NSS/SCL/HSU_RX1, PA5/RSTPD_N1, PA7/IRQ1, PC1, PC2, PC3, RX1, TX1, TX2: TestPoint, TestPoint:TestPoint_Pad_D1.0mm, symbol Connector:TestPoint
Connections:
- net +3.3V: now also DVDD1.1, I1.1
- net +BAT: now also +BAT1.1
- net GND: now also GND1.1
- net PA1: now also PA1/MOSI/SDA/HSU_TX1.1
- net PA2: now also PA2/MISO/P71.1
- net PA3: now also PA3/SCK/P72.1
- net PA4: now also PA4/NSS/SCL/HSU_RX1.1
- net PA5: now also PA5/RSTPD_N1.1
- net PA7: now also PA7/IRQ1.1
- net PC1: now also PC1.1
- net PC2: now also PC2.1
- net PC3: now also PC3.1
- net RX: now also RX1.1
- net TX1: now also TX1.1
- net TX2: now also TX2.1
- net at R10.2, U2.16 (I0): now also I0.1
Other:
- moved on the sheet: R10

Commit message: Fixes To SCH, 4-Layer PCB In Progress
Parts:
- removed H1, H2, H3, H4: MountingHole, MountingHole:MountingHole_2.2mm_M2, symbol Mechanical:MountingHole
- removed J2, J3: Conn_02x20_Counter_Clockwise, symbol Connector_Generic:Conn_02x20_Counter_Clockwise
- added H1, H2, H3, H4: MountingHole_Pad, MountingHole:MountingHole_2.2mm_M2_Pad, symbol Mechanical:MountingHole_Pad
Connections:
- net +3.3V: now also C16.1, C18.1, C19.1, U2.23 (PVDD), U3.1 (VCC)
- net GND: now also H1.1, H2.1, H3.1, H4.1
- net VCC: no longer C16.1, C18.1, C19.1, U2.23 (PVDD), U3.1 (VCC)

Commit message: Updated Sch, Traces Routed, Needs Verification
Parts:
- removed R3: 4.7k, Resistor_SMD:R_0805_2012Metric_Pad1.20x1.40mm_HandSolder, symbol Device:R_Small_US
- removed SW2: SW_DPDT_x2, Button_Switch_THT:SW_CK_JS202011CQN_DPDT_Straight, symbol Switch:SW_DPDT_x2
- added J2, J3: READ/WRITE, Connector_PinHeader_2.54mm:PinHeader_1x03_P2.54mm_Vertical, symbol Connector_Generic:Conn_01x03
Connections:
- net +3.3V: no longer C14.1, C15.1, C7.1, C8.1, C9.1, DVDD1.1, I1.1, U2.17 (I1), U2.39 (DVDD), U2.5 (TVDD), U2.8 (AVDD)
- net PA0: now also J2.3 (Pin_3)
- net PB2: now also J2.1 (Pin_1)
- net PB3: now also J3.1 (Pin_1)
- net at D1.1 (K): now also J3.3 (Pin_3)
- net at J12.2 (Pin_2): now also J2.2 (Pin_2)
- net at J12.3 (Pin_3): now also J3.2 (Pin_2)
- new net AVDD: C8.1, U2.8 (AVDD)
- new net DVDD: C14.1, C15.1, DVDD1.1, I1.1, U2.17 (I1), U2.39 (DVDD)
- new net TVDD: C7.1, C9.1, U2.5 (TVDD)

Commit message: Antenna Fix + DRC Fixes
Connections:
- new net: C1.1, C3.1, J4.3 (Pin_3)
- new net: C1.2, C2.1, C5.2, C6.1, J4.2 (Pin_2)
- new net: C2.2, C4.1, J4.1 (Pin_1)
Changed lines of the file:
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@@
-	)
-	(junction
-		(at 34.29 140.97)
-		(diameter 0)
-		(color 0 0 0 0)
 	)
 	(junction
@@
 	)
 	(junction
-		(at 34.29 138.43)
-		(diameter 0)
-		(color 0 0 0 0)
-	)
-	(junction
 		(at 60.96 123.19)
 		(diameter 0)
@@
 	)
 	(junction
-		(at 34.29 135.89)
-		(diameter 0)
-		(color 0 0 0 0)
-	)
-	(junction
 		(at 215.9 34.29)
 		(diameter 0)
@@
 	(wire
 		(pts
-			(xy 34.29 138.43) (xy 34.29 140.97)
-		)
-		(stroke
-			(width 0)
-			(type default)
-		)
-	)
-	(wire
-		(pts
 			(xy 173.99 40.64) (xy 187.96 40.64)
 		)
@@
 		(pts
 			(xy 36.83 220.98) (xy 36.83 231.14)
-		)
-		(stroke
-			(width 0)
-			(type default)
-		)
-	)
-	(wire
-		(pts
-			(xy 34.29 135.89) (xy 34.29 138.43)
 		)
 		(stroke
@@
 		)
 		(fill
+			(type none)
+		)
+	)
+	(rectangle
+		(start 223.52 49.53)
+		(end 252.73 77.47)
+		(stroke
+			(width 0.508)
+			(type default)
+			(color 255 131 123 1)
+		)
+		(fill

Commit message: Tracewidth Fixes
Changed lines of the file:
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@@
-	)
-	(rectangle
-		(start 223.52 49.53)
-		(end 252.73 77.47)
-		(stroke
-			(width 0.508)
-			(type default)
-			(color 255 131 123 1)
-		)
-		(fill
-			(type none)
-		)
 	)
 	(rectangle
