File: Schematics & PCB/sensOrb/salp_board_round.kicad_pcb (KiCad board)
At the start: 4 copper layers, 135.6 x 58.7 mm, 61 parts, among them J1 ATTINY3226, J10 POWER, J2 READ/WRITE, J3 READ/WRITE, J4 Conn_01x03, J8 ATTINY3226, J9 POWER_JUMPER, Q1 IRLML6402, Q2 IRLML6402, U1 LD1117S33TR, U2 PN5321A3HN/C106_55, U3 ATtiny3226-S, U4 TP4057, U6 DW01A, Y2 27.12 MHz

Commit message: PCB Layout Initializing
Parts:
- removed H3, H4: MountingHole_Pad, MountingHole:MountingHole_2.2mm_M2_Pad
- removed J12: ~, Connector_PinHeader_2.54mm:PinHeader_1x06_P2.54mm_Horizontal
- removed J2: READ/WRITE, Connector_PinHeader_2.54mm:PinHeader_1x03_P2.54mm_Vertical
- removed U6: DW01A, Package_TO_SOT_SMD:SOT-23-6
- removed Y2: 27.12 MHz, Crystal:Crystal_SMD_SeikoEpson_TSX3225-4Pin_3.2x2.5mm_HandSoldering
- added D6: LED, LED_SMD:LED_0603_1608Metric_Pad1.05x0.95mm_HandSolder, F.Cu at (120.5, 83.4)
- added J5: ATTINY3226, Connector_PinSocket_2.54mm:PinSocket_2x09_P2.54mm_Vertical, F.Cu at (90.0, 63.7)
- added J6: ~, Connector_PinHeader_2.54mm:PinHeader_1x06_P2.54mm_Vertical, F.Cu at (115.0, 63.7)
- added J7: READ/WRITE, Connector_PinHeader_2.54mm:PinHeader_1x03_P2.54mm_Vertical, F.Cu at (99.3, 110.2)
- added R12: 560, Resistor_SMD:R_0805_2012Metric_Pad1.20x1.40mm_HandSolder, F.Cu at (89.9, 96.6)
- added R3: 1K, Resistor_SMD:R_0805_2012Metric_Pad1.20x1.40mm_HandSolder, F.Cu at (80.4, 99.6)
- added U5: DW01A, Package_TO_SOT_SMD:SOT-23-6, F.Cu at (130.2, 114.9)
- added Y1: 27.12 MHz, Crystal:Crystal_SMD_SeikoEpson_TSX3225-4Pin_3.2x2.5mm_HandSoldering, F.Cu at (129.6, 101.9)
- C1, C2: value 200p -> 100 nF
- C10: value .1u -> 22p
- C11: value 1n -> 4.7uF
- C12, C13: value 22pF -> 220p
- C14: value 100 nF -> 1uF
- C15: value 10uF -> 22pF
- C16: value 10nF -> .1u
- C17: value 10 uF -> 1n
- C18: value 100nF -> 22pF
- C19: value 1uF -> 100nF
- C20: value 100nF -> 10uF
- C21: value 100nF -> 0.1 uF
- C22: value 10uF -> 100nF
- C23: value 0.1 uF -> 10 uF
- C3: value 22p -> 4.7uF
- C4: value 22p -> 10nF
- C5, C6: value 220p -> 200p
- C7: value .1u -> 100nF
- C8: value 100 nF -> 100nF
- C9: value 4.7u -> 22p
- D1: value BZS55C5V1 -> APFA3010; footprint Diode_SMD:D_1206_3216Metric_Pad1.42x1.75mm_HandSolder -> LED_SMD:LED_Kingbright_APFA3010_3x1.5mm_Horizontal
- D2: value LED -> BZS55C5V1; footprint LED_SMD:LED_0805_2012Metric -> Diode_SMD:D_1206_3216Metric_Pad1.42x1.75mm_HandSolder
- D4: value BAT54CW -> LED; footprint Package_TO_SOT_SMD:SOT-323_SC-70 -> LED_SMD:LED_0805_2012Metric
- D5: value APFA3010 -> BAT54CW; footprint LED_SMD:LED_Kingbright_APFA3010_3x1.5mm_Horizontal -> Package_TO_SOT_SMD:SOT-323_SC-70
- J1: value ATTINY3226 -> Antenna; footprint Connector_PinSocket_2.54mm:PinSocket_2x09_P2.54mm_Vertical -> Connector_PinHeader_2.54mm:PinHeader_1x03_P2.54mm_Vertical
- J10: value POWER -> COMM_SEL_0; footprint Connector_PinSocket_2.54mm:PinSocket_2x03_P2.54mm_Vertical -> Connector_PinHeader_2.54mm:PinHeader_1x03_P2.54mm_Vertical
- J3: value READ/WRITE -> ATTINY3226; footprint Connector_PinHeader_2.54mm:PinHeader_1x03_P2.54mm_Vertical -> Connector_PinSocket_2.54mm:PinSocket_2x09_P2.54mm_Vertical
- J4: value Conn_01x03 -> POWER; footprint Connector_PinHeader_2.54mm:PinHeader_1x03_P2.54mm_Horizontal -> Connector_PinSocket_2.54mm:PinSocket_2x03_P2.54mm_Vertical
- J8: value ATTINY3226 -> READ/WRITE; footprint Connector_PinSocket_2.54mm:PinSocket_2x09_P2.54mm_Vertical -> Connector_PinHeader_2.54mm:PinHeader_1x03_P2.54mm_Vertical
- J9: value POWER_JUMPER -> COMM_SEL_1
- R1: value 1.6K -> 1k
- R10: value 1k -> 3.9k
- R11: value 100 -> 1k
- R2: value 1K -> 2.7K
- R4: value 1k -> 10
- R5: value 3.9k -> 10
- R6: value 10 -> 68
- R7: value 10 -> 100
- R8: value 68 -> 1k
- U1: value LD1117S33TR -> PN5321A3HN/C106_55; footprint Package_TO_SOT_SMD:SOT-223-3_TabPin2 -> PN532:QFN40G-0.5-6X6MM
- U2: value PN5321A3HN/C106_55 -> ATtiny3226-S; footprint PN532:QFN40G-0.5-6X6MM -> Package_SO:SOIC-20W_7.5x12.8mm_P1.27mm
- U3: value ATtiny3226-S -> TP4057; footprint Package_SO:SOIC-20W_7.5x12.8mm_P1.27mm -> Package_TO_SOT_SMD:TSOT-23-6
- U4: value TP4057 -> LD1117S33TR; footprint Package_TO_SOT_SMD:TSOT-23-6 -> Package_TO_SOT_SMD:SOT-223-3_TabPin2
- moved J3 106.3 mm to (82.9, 63.7), turned to 0 degrees
- moved U2 94.8 mm to (84.5, 108.3)
- moved L1 90.5 mm to (80.4, 87.8), turned to 0 degrees
- moved R10 90.3 mm to (89.9, 90.7), turned to 0 degrees
- moved J10 88.0 mm to (113.3, 110.2)
- moved J8 86.9 mm to (104.0, 110.2), turned to 0 degrees
- moved R2 86.6 mm to (80.4, 96.6), turned to 0 degrees
- moved H2 85.9 mm to (109.7, 70.3)
- moved L2 85.7 mm to (80.4, 90.7)
- moved C20 82.2 mm to (104.4, 71.9), turned to 0 degrees
- moved J1 81.7 mm to (94.7, 110.2)
- moved C16 78.7 mm to (99.5, 83.9)
- moved D1 78.7 mm to (115.5, 80.7)
- moved R1 78.0 mm to (80.4, 93.7)
- moved R4 77.0 mm to (85.2, 87.8), turned to 0 degrees
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Connections:
- C1 pad 1: Net-(J4-Pin_3) -> /AVDD
- C1 pad 2: Net-(J4-Pin_2) -> GND
- C10 pad 1: /VMID -> Net-(J1-Pin_1)
- C10 pad 2: GND -> Net-(C10-Pad2)
- C11 pad 1: Net-(C11-Pad1) -> /AVDD
- C11 pad 2: /RX -> GND
- C12 pad 1: /OSCIN -> Net-(C12-Pad1)
- C12 pad 2: GND -> Net-(J1-Pin_2)
- C13 pad 1: /OSCOUT -> Net-(J1-Pin_2)
- C13 pad 2: GND -> Net-(C10-Pad2)
- C14 pad 1: /DVDD -> +3.3V
- C15 pad 1: /DVDD -> /OSCIN
- C16 pad 1: +3.3V -> /VMID
- C17 pad 1: GND -> Net-(C17-Pad1)
- C17 pad 2: +BAT -> /RX
- C18 pad 1: +3.3V -> /OSCOUT
- C19 pad 1: +3.3V -> GND
- C19 pad 2: GND -> +3.3V
- C2 pad 1: Net-(J4-Pin_2) -> /AVDD
- C2 pad 2: Net-(J4-Pin_1) -> GND
- C21 pad 1: VCC -> GND
- C21 pad 2: GND -> Net-(U5-VCC)
- C22 pad 1: /V_REG -> VCC
- C23 pad 2: Net-(U6-VCC) -> +BAT
- C3 pad 1: Net-(J4-Pin_3) -> /AVDD
- C3 pad 2: Net-(C3-Pad2) -> GND
- C4 pad 1: Net-(J4-Pin_1) -> +3.3V
- C4 pad 2: Net-(C4-Pad2) -> GND
- C5 pad 1: Net-(C3-Pad2) -> Net-(J1-Pin_3)
- C5 pad 2: Net-(J4-Pin_2) -> Net-(J1-Pin_2)
- C6 pad 1: Net-(J4-Pin_2) -> Net-(J1-Pin_2)
- C6 pad 2: Net-(C4-Pad2) -> Net-(J1-Pin_1)
- C7 pad 1: /TVDD -> /AVDD
- C8 pad 1: /AVDD -> +3.3V
- C9 pad 1: /TVDD -> Net-(J1-Pin_3)
- C9 pad 2: GND -> Net-(C12-Pad1)
- D1 pad 1: Net-(D1-K) -> Net-(D1-R)
- D1 pad 2: /PA0 -> GND
- D2 pad 2: Net-(D2-A) -> /PA0
- D3 pad 2: Net-(D2-A) -> Net-(D3-A)
- D4 pad 1: +BAT -> Net-(D4-K)
- D4 pad 2: /V_USB -> Net-(D3-A)
- D5 pad 1: Net-(D5-R) -> +BAT
- D5 pad 2: GND -> /V_USB
- D5 pad 3: Net-(D5-G) -> VCC
- J1 pad 1: /PA4 -> Net-(J1-Pin_1)
- J1 pad 2: /PA4 -> Net-(J1-Pin_2)
- J1 pad 3: /PA5 -> Net-(J1-Pin_3)
- J10 pad 1: VCC -> GND
- J10 pad 2: GND -> Net-(J10-Pin_2)
- J10 pad 3: GND -> /AVDD
- J3 pad 1: /PB3 -> /M_SCL
- J3 pad 2: Net-(J12-Pin_3) -> /M_SCL
- J3 pad 3: Net-(D1-K) -> /PA5
- J4 pad 1: Net-(J4-Pin_1) -> VCC
- J4 pad 2: Net-(J4-Pin_2) -> GND
- J4 pad 3: Net-(J4-Pin_3) -> GND
- J8 pad 1: /M_SCL -> /PB3
- J8 pad 2: /M_SCL -> Net-(J6-Pin_3)
- J8 pad 3: /PC0 -> Net-(D2-K)
- J9 pad 1: /VOR -> GND
- J9 pad 2: +3.3V -> Net-(J9-Pin_2)
- J9 pad 3: /V_REG -> /AVDD
- L1 pad 1: Net-(C3-Pad2) -> Net-(C12-Pad1)
- L2 pad 1: Net-(C4-Pad2) -> Net-(C10-Pad2)
- R1 pad 1: Net-(C4-Pad2) -> Net-(J9-Pin_2)
- R1 pad 2: Net-(C11-Pad1) -> /I1
- R10 pad 2: Net-(U2-I0) -> Net-(U3-PROG)
- R11 pad 1: +BAT -> Net-(J10-Pin_2)
- R11 pad 2: Net-(U6-VCC) -> /I0
- R2 pad 1: /VMID -> Net-(C10-Pad2)
- R2 pad 2: /RX -> Net-(C17-Pad1)
- R4 pad 1: Net-(D2-A) -> Net-(D1-B)
- R4 pad 2: /V_USB -> /PC1
- R5 pad 1: GND -> Net-(D1-G)
- R5 pad 2: Net-(U4-PROG) -> /PC2
- R6 pad 1: Net-(D5-B) -> Net-(D1-R)
- R6 pad 2: /PC1 -> /PC3
- R7 pad 1: Net-(D5-G) -> +BAT
- R7 pad 2: /PC2 -> Net-(U5-VCC)
- R8 pad 1: Net-(D5-R) -> GND
- R8 pad 2: /PC3 -> Net-(U5-CS)
- R9 pad 1: GND -> Net-(D3-A)
- R9 pad 2: Net-(U6-CS) -> /V_USB
- U1 pad 2: /V_REG -> unconnected-(U1-LOADMOD-Pad2)
- U1 pad 3: VCC -> GND
- U2 pad 1: GND -> +3.3V
- U2 pad 10: /RX -> /M_SCL
- U2 pad 11: GND -> /M_SCL
- U2 pad 12: unconnected-(U2-AUX1-Pad12) -> /PC0
- U2 pad 13: unconnected-(U2-AUX2-Pad13) -> /PC1
- U2 pad 14: /OSCIN -> /PC2
- U2 pad 15: /OSCOUT -> /PC3
- U2 pad 16: Net-(U2-I0) -> /PA0
- U2 pad 17: /DVDD -> /M_SCL
- U2 pad 18: GND -> /M_SCL
- U2 pad 19: unconnected-(U2-P35-Pad19) -> /PA3
- U2 pad 2: unconnected-(U2-LOADMOD-Pad2) -> /M_SCL
- U2 pad 20: unconnected-(U2-N.C.-Pad20) -> GND
- U2 pad 3: GND -> /PA5
- U2 pad 4: /TX1 -> /PA6
- U2 pad 5: /TVDD -> /PA7
- U2 pad 6: /TX2 -> /PB5
- U2 pad 7: GND -> /PB4
- U2 pad 8: /AVDD -> /PB3
- U2 pad 9: /VMID -> /PB2
- U3 pad 1: +3.3V -> Net-(D3-K)
- U3 pad 2: /PA4 -> GND
- U3 pad 3: /PA5 -> +BAT
- U3 pad 4: /PA6 -> /V_USB
- U3 pad 5: /PA7 -> Net-(D4-K)
- U3 pad 6: /PB5 -> Net-(U3-PROG)
- U4 pad 1: Net-(D2-K) -> GND
- U4 pad 2: GND -> +3.3V
- U4 pad 3: +BAT -> VCC
Routing:
- net +BAT: track 96.5 -> 0.00 mm, vias 3 -> 0
- net GND: track 89.4 -> 0.00 mm, vias 24 -> 0
- net VCC: track 78.6 -> 0.00 mm, vias 1 -> 0
- net /V_USB: track 62.8 -> 0.00 mm, vias 2 -> 0
- net /PC3: track 50.1 -> 0.00 mm, vias 2 -> 0
- net /PC1: track 47.7 -> 0.00 mm, vias 2 -> 0
- net /PC2: track 47.6 -> 0.00 mm, vias 2 -> 0
- net /PA1: track 37.0 -> 0.00 mm
- net /PA2: track 35.7 -> 0.00 mm, vias 1 -> 0
- net /PA3: track 34.9 -> 0.00 mm
- net /OSCOUT: track 34.6 -> 0.00 mm
- net /PA7: track 31.2 -> 0.00 mm, vias 1 -> 0
- net /PA5: track 30.4 -> 0.00 mm, vias 1 -> 0
- net /PA0: track 30.3 -> 0.00 mm, vias 2 -> 0
- net /PA4: track 26.9 -> 0.00 mm, vias 1 -> 0
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- added copper zone on In2.Cu, net +3.3V
- added copper zone on In1.Cu, net GND
- removed copper zone on In1.Cu, net +3.3V
- removed copper zone on In2.Cu, net GND
Other:
- board size 135.6 x 58.7 mm -> 56.2 x 56.2 mm
- board text removed: "For use with a 3.7V 500 mAH LiOn or Li-Po coin cell battery"
- board text removed: "Initial Design by Owen Pyle Revisions by Jack Cunningham 6/23/25"
- board text removed: "LEFT-Monitor RIGHT-Program"
- board text removed: "PA0"
- board text removed: "PA1"
- board text removed: "PA2"
- board text removed: "PA3"
- board text removed: "PA4"
- board text removed: "PA5"
- board text removed: "PA6"
- board text removed: "PA7"
- board text removed: "PB2"
- board text removed: "PB3"
- board text removed: "PB4"
- board text removed: "PB5"
- board text removed: "PC0"
- board text removed: "PC1"
- board text removed: "PC2"
- board text removed: "PC3"
- board text removed: "PN532 ATTINY3226 NODE DEMO BOARD V2"
- board text removed: "SCL"
- board text removed: "SDA"

Commit message: PCB Progress
Parts:
- moved H1 78.8 mm to (170.0, 115.1)
- moved H2 60.5 mm to (170.0, 64.9)
- moved J6 4.14 mm to (110.9, 63.8)
Changed lines of the file:
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@@
 	(footprint "Connector_PinHeader_2.54mm:PinHeader_1x06_P2.54mm_Vertical"
 		(layer "F.Cu")
-		(at 115.0375 63.66)
+		(at 110.9 63.76)
 		(descr "Through hole straight pin header, 1x06, 2.54mm pitch, single row")
 		(tags "Through hole pin header THT 1x06 2.54mm single row")
@@
 	(footprint "MountingHole:MountingHole_2.2mm_M2_Pad"
 		(layer "F.Cu")
-		(at 109.7375 70.26)
+		(at 170 64.9)
 		(descr "Mounting Hole 2.2mm, M2")
 		(tags "mounting hole 2.2mm m2")
 		(property "Reference" "H2"
-			(at 0 -3.2 0)
+			(at 3.8 -1.4 0)
 			(layer "F.SilkS")
 			(effects
@@
 		)
 		(property "Value" "MountingHole_Pad"
-			(at 0 3.2 0)
+			(at 0 -3.9 0)
 			(layer "F.Fab")
 			(effects
@@
 	(footprint "MountingHole:MountingHole_2.2mm_M2_Pad"
 		(layer "F.Cu")
-		(at 109.7375 64.31)
+		(at 170 115.1)
 		(descr "Mounting Hole 2.2mm, M2")
 		(tags "mounting hole 2.2mm m2")

Commit message: PCB Design Progress
Parts:
- moved U1 15.3 mm to (115.5, 91.3)
Changed lines of the file:
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@@
 	(footprint "PN532:QFN40G-0.5-6X6MM"
 		(layer "F.Cu")
-		(at 130.7115 89.265)
+		(at 115.5 91.3)
 		(property "Reference" "U1"
 			(at 0.318118 -4.262798 0)

Commit message: PCB Layout Progress
Parts:
- D5, Q1, Q2, U3, U5: moved to B.Cu
- moved J3 111.2 mm to (192.7, 81.3), turned to -90 degrees
- moved U2 102.5 mm to (185.3, 89.5), turned to -90 degrees
- moved J6 99.8 mm to (208.5, 84.8)
- moved J5 89.8 mm to (173.1, 97.8), turned to 90 degrees
- moved J8 88.0 mm to (184.5, 74.6), turned to 90 degrees
- moved J7 83.5 mm to (174.9, 74.6), turned to 90 degrees
- moved J9 68.9 mm to (162.5, 67.3)
- moved J10 68.5 mm to (166.7, 67.3)
- moved J4 63.2 mm to (183.4, 104.4), turned to 90 degrees
- moved J1 57.2 mm to (146.3, 85.5), turned to 180 degrees
- moved U4 52.0 mm to (176.3, 106.3), turned to 180 degrees
- moved U1 42.5 mm to (157.3, 84.2)
- moved U3 37.2 mm to (166.8, 103.7)
- moved Q2 36.5 mm to (161.3, 109.2), turned to 180 degrees
- moved H1 35.5 mm to (144.9, 90.0)
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Other:
- outline, holes or cut-outs redrawn

Commit message: Routing Progress
Parts:
- C21, C23, D1, D3, D4, R10, R4, R5, R6, R7, R8, R9: moved to B.Cu
- moved C8 83.9 mm to (192.3, 85.3), turned to -90 degrees
- moved C14 82.0 mm to (195.3, 85.3), turned to -90 degrees
- moved C4 80.9 mm to (189.0, 85.3), turned to -90 degrees
- moved R5 80.3 mm to (178.7, 104.7), turned to 90 degrees
- moved R4 78.5 mm to (176.5, 104.7), turned to 90 degrees
- moved R12 77.6 mm to (180.6, 111.7)
- moved R6 75.5 mm to (174.2, 104.7), turned to 90 degrees
- moved R1 69.2 mm to (156.9, 69.6), turned to -90 degrees
- moved C20 67.0 mm to (173.7, 114.4)
- moved R11 66.6 mm to (163.5, 69.5), turned to -90 degrees
- moved R10 65.2 mm to (167.8, 107.6), turned to 90 degrees
- moved C22 63.8 mm to (175.1, 111.8), turned to 180 degrees
- moved R3 63.5 mm to (156.0, 90.3)
- moved L1 62.6 mm to (156.0, 102.9), turned to 90 degrees
- moved R9 60.1 mm to (162.6, 104.6), turned to 90 degrees
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Routing:
- net GND: track 0.00 -> 106.2 mm, vias 0 -> 19
- net VCC: track 0.00 -> 54.3 mm
- net /M_SCL: track 0.00 -> 51.2 mm
- net /PA0: track 0.00 -> 49.4 mm
- net /AVDD: track 0.00 -> 41.4 mm, vias 0 -> 2
- net +3.3V: track 0.00 -> 37.0 mm, vias 0 -> 6
- net /V_USB: track 0.00 -> 30.6 mm
- net +BAT: track 0.00 -> 30.5 mm, vias 0 -> 5
- net Net-(J1-Pin_2): track 0.00 -> 25.8 mm
- net /I1: track 0.00 -> 23.6 mm, vias 0 -> 2
- net /I0: track 0.00 -> 23.1 mm, vias 0 -> 2
- net /TX1: track 0.00 -> 21.3 mm, vias 0 -> 2
- net Net-(J6-Pin_3): track 0.00 -> 20.9 mm
- net Net-(J1-Pin_1): track 0.00 -> 20.1 mm, vias 0 -> 1
- net /PC3: track 0.00 -> 19.9 mm
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
Commit message: Routing Progress
Parts:
- moved C19 1.14 mm to (163.0, 86.9), turned to 90 degrees
Routing:
- net Net-(D6-A): track 0.00 -> 2.24 mm
- net +3.3V: track 37.0 -> 35.7 mm
- net GND: track 106.2 -> 105.3 mm
Changed lines of the file:
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@@
 	)
 	(paper "A4")
+	(title_block
+		(date "2025-07-02")
+	)
 	(layers
 		(0 "F.Cu" signal "Front_Signal")
@@
 	(footprint "Capacitor_SMD:C_0805_2012Metric_Pad1.18x1.45mm_HandSolder"
 		(layer "F.Cu")
-		(at 163.7 86 180)
+		(at 163 86.9 90)
 		(descr "Capacitor SMD 0805 (2012 Metric), square (rectangular) end terminal, IPC_7351 nominal with elongated pad for handsoldering. (Body size source: IPC-SM-782 page 76, https://www.pcb-3d.com/wordpress/wp-content/uploads/ipc-sm-782a_amendment_1_and_2.pdf, https://docs.google.com/spreadsheets/d/1BsfQQcO9C6DZCsRaXUlFlo91Tg2WpOkGARC1WS5S8t0/edit?usp=sharing), generated with kicad-footprint-generator")
 		(tags "capacitor handsolder")
 		(property "Reference" "C19"
-			(at 0 -1.68 360)
+			(at 0 -1.68 90)
 			(layer "F.SilkS")
 			(effects
@@
 		)
 		(property "Value" "100nF"
-			(at 0 1.68 360)
+			(at 0 1.68 90)
 			(layer "F.Fab")
 			(effects
@@
 		)
 		(property "Footprint" "Capacitor_SMD:C_0805_2012Metric_Pad1.18x1.45mm_HandSolder"
-			(at 0 0 180)
+			(at 0 0 90)
 			(unlocked yes)
 			(layer "F.Fab")
@@
 		)
 		(property "Datasheet" ""
-			(at 0 0 180)
+			(at 0 0 90)
 			(unlocked yes)
 			(layer "F.Fab")
@@
 		)
 		(property "Description" "Unpolarized capacitor"
-			(at 0 0 180)
+			(at 0 0 90)
 			(unlocked yes)
 			(layer "F.Fab")
@@
 		(attr smd)
 		(fp_line
-			(start -0.261252 0.735)
-			(end 0.261252 0.735)
+			(start -0.261252 -0.735)
+			(end 0.261252 -0.735)
 			(stroke
 				(width 0.12)
@@
 		)
 		(fp_line
-			(start -0.261252 -0.735)
-			(end 0.261252 -0.735)
+			(start -0.261252 0.735)
+			(end 0.261252 0.735)
 			(stroke
 				(width 0.12)
@@
 		)
 		(fp_line
-			(start 1.88 0.98)
-			(end -1.88 0.98)
+			(start 1.88 -0.98)
+			(end 1.88 0.98)
 			(stroke
 				(width 0.05)
@@
 		)
 		(fp_line
-			(start 1.88 -0.98)
-			(end 1.88 0.98)
+			(start -1.88 -0.98)
+			(end 1.88 -0.98)
 			(stroke
 				(width 0.05)
@@
 		)
 		(fp_line
-			(start -1.88 0.98)
-			(end -1.88 -0.98)
+			(start 1.88 0.98)
+			(end -1.88 0.98)
 			(stroke
 				(width 0.05)
@@
 		)
 		(fp_line
-			(start -1.88 -0.98)
-			(end 1.88 -0.98)
+			(start -1.88 0.98)
+			(end -1.88 -0.98)
 			(stroke
 				(width 0.05)
@@
 		)
 		(fp_line
-			(start 1 0.625)
-			(end -1 0.625)
+			(start 1 -0.625)
+			(end 1 0.625)
 			(stroke
 				(width 0.1)
@@
 		)
 		(fp_line
-			(start 1 -0.625)
-			(end 1 0.625)
+			(start -1 -0.625)
+			(end 1 -0.625)
 			(stroke
 				(width 0.1)
@@
 		)
 		(fp_line
-			(start -1 0.625)
-			(end -1 -0.625)
+			(start 1 0.625)
+			(end -1 0.625)
 			(stroke
 				(width 0.1)
@@
 		)
 		(fp_line
-			(start -1 -0.625)
-			(end 1 -0.625)
+			(start -1 0.625)
+			(end -1 -0.625)
 			(stroke
 				(width 0.1)
@@
 		)
 		(fp_text user "${REFERENCE}"
-			(at 0 0 360)
+			(at 0 0 90)
 			(layer "F.Fab")
 			(effects
@@
 		)
 		(pad "1" smd roundrect
-			(at -1.0375 0 180)
+			(at -1.0375 0 90)
 			(size 1.175 1.45)
 			(layers "F.Cu" "F.Paste" "F.Mask")
@@
 		)
 		(pad "2" smd roundrect
-			(at 1.0375 0 180)
+			(at 1.0375 0 90)
 			(size 1.175 1.45)
 			(layers "F.Cu" "F.Paste" "F.Mask")
@@
 	)
 	(segment
-		(start 166.2 87.3)
-		(end 166.1 87.2)
-		(width 0.2)
-		(layer "F.Cu")
-		(net 1)
-	)
-	(segment
 		(start 154.4 81.9)
 		(end 154 81.5)
@@
 	)
 	(segment
-		(start 166.1 87.3)
-		(end 166.2 87.3)
-		(width 0.2)
-		(layer "F.Cu")
-		(net 1)
-	)
-	(segment
 		(start 192.2625 86.3375)
 		(end 192.3 86.3)
@@
 	)
 	(segment
+		(start 163 87.9375)
+		(end 163 89.2)
+		(width 0.2)
+		(layer "F.Cu")
+		(net 1)
+	)
+	(segment
 		(start 156.6 84.9)
 		(end 157.35 84.15)
@@
 	)
 	(segment
+		(start 163 89.2)
+		(end 163 89.1)
+		(width 0.2)
+		(layer "F.Cu")
+		(net 1)
+	)
+	(segment
 		(start 166.7 100.2875)
 		(end 166.8875 100.2875)
@@
 	)
 	(segment
-		(start 166.1 87.2)
-		(end 166.1 87.3)
-		(width 0.2)
-		(layer "F.Cu")
-		(net 1)
-	)
-	(segment
 		(start 167.6 92)
 		(end 167.7 92)
@@
 	)
 	(segment
-		(start 164.7375 86)
-		(end 164.9 86)
-		(width 0.2)
-		(layer "F.Cu")
-		(net 1)
-	)
-	(segment
 		(start 166.7 100.2875)
 		(end 166.3125 100.2875)
@@
 		(net 1)
 	)
-	(segment
-		(start 164.9 86)
-		(end 166.1 87.2)
-		(width 0.2)
-		(layer "F.Cu")
-		(net 1)
-	)
 	(via
 		(at 191.1 88.8)
@@
 	)
 	(via
-		(at 167.7 92)
+		(at 163 89.2)
 		(size 0.6)
 		(drill 0.3)
@@
 	)
 	(via
-		(at 167.9 110.3)
+		(at 167.7 92)
 		(size 0.6)
 		(drill 0.3)
@@
 	)
 	(via
-		(at 176 115.9)
+		(at 167.9 110.3)
 		(size 0.6)
 		(drill 0.3)
@@
 	)
 	(via
-		(at 181.3 109.3)
+		(at 176 115.9)
 		(size 0.6)
 		(drill 0.3)
@@
 	)
 	(via
-		(at 166.1 87.3)
+		(at 181.3 109.3)
 		(size 0.6)
 		(drill 0.3)
@@
 	)
 	(segment
-		(start 157.2 88.9)
-		(end 157.1 88.8)
+		(start 166.7 95.7375)
+		(end 165.3625 94.4)
 		(width 0.2)
 		(layer "F.Cu")
@@
 	)
 	(segment
-		(start 166.7 95.7375)
-		(end 165.3625 94.4)
+		(start 162.7 94.4)
+		(end 161.7 93.4)
 		(width 0.2)
 		(layer "F.Cu")
@@
 	)
 	(segment
-		(start 161.7 92.84957)
-		(end 157.75043 88.9)
+		(start 157.1 88.2)
+		(end 157.1 87.1)
 		(width 0.2)
 		(layer "F.Cu")
@@
 	(segment
 		(start 161.7 93.4)
-		(end 161.7 92.84957)
+		(end 161.7 92.6)
 		(width 0.2)
 		(layer "F.Cu")
@@
 	)
 	(segment
-		(start 157.1 88.8)
-		(end 157.1 87.1)
+		(start 161.7 92.6)
+		(end 157.95043 88.85043)
 		(width 0.2)
 		(layer "F.Cu")
@@
 	)
 	(segment
-		(start 162.7 94.4)
-		(end 161.7 93.4)
+		(start 157.95043 88.85043)
+		(end 157.75043 88.85043)
 		(width 0.2)
 		(layer "F.Cu")
@@
 	)
 	(segment
-		(start 157.75043 88.9)
-		(end 157.2 88.9)
+		(start 157.75043 88.85043)
+		(end 157.1 88.2)
 		(width 0.2)
 		(layer "F.Cu")
@@
 	)
 	(segment
-		(start 162.6625 86)
-		(end 162.0625 85.4)
-		(width 0.2)
-		(layer "F.Cu")
-		(net 8)
-	)
-	(segment
 		(start 154.6 80.5)
 		(end 154.7 80.6)
@@
 	)
 	(segment
-		(start 162.0625 85.4)
-		(end 160.3 85.4)
-		(width 0.2)
-		(layer "F.Cu")
-		(net 8)
-	)
-	(segment
 		(start 186.315 84.55)
 		(end 188.7125 84.55)
@@
 	)
 	(segment
-		(start 162.6625 86)
-		(end 162.6625 87.5625)
+		(start 162.5375 85.4)
+		(end 163 85.8625)
 		(width 0.2)
 		(layer "F.Cu")
@@
 	)
 	(segment
-		(start 162.7 87.6)
-		(end 162.6625 87.5625)
+		(start 160.3 85.4)
+		(end 161.5 85.4)
+		(width 0.2)
+		(layer "F.Cu")
+		(net 8)
+	)
+	(segment
+		(start 161.5 85.4)
+		(end 162.5375 85.4)
 		(width 0.2)
 		(layer "F.Cu")
@@
 	)
 	(via
-		(at 185.9 109.6)
+		(at 161.5 85.4)
 		(size 0.6)
 		(drill 0.3)
@@
 	)
 	(via
-		(at 154.6 80.5)
+		(at 185.9 109.6)
 		(size 0.6)
 		(drill 0.3)
@@
 	)
 	(via
-		(at 162.7 87.6)
+		(at 154.6 80.5)
 		(size 0.6)
 		(drill 0.3)
@@
 	)
 	(segment
+		(start 181.5 113.9)
+		(end 181.5 111.8)
+		(width 0.2)
+		(layer "F.Cu")
+		(net 43)
+	)
+	(segment
+		(start 181.5 111.8)
+		(end 181.6 111.7)
+		(width 0.2)
+		(layer "F.Cu")
+		(net 43)
+	)
+	(segment

Commit message: All Routed
To do: Verify electrical connections(do they make sense), trace widths, DRC violations
Parts:
- moved C19 2.06 mm to (161.9, 88.6)
Routing:
- net /M_SCL: track 51.2 -> 109.7 mm, vias 0 -> 4
- net /PA5: track 12.1 -> 48.5 mm, vias 0 -> 1
- net /PA3: track 13.1 -> 46.4 mm, vias 0 -> 2
- net /PA7: track 8.09 -> 30.7 mm
- net /PB5: track 4.67 -> 7.21 mm
- net /PA0: track 49.4 -> 51.5 mm

Commit message: Various Tracewidth Adjustments, DRC Fixes
Routing:
- net VCC: track 54.3 -> 56.1 mm
- net /V_USB: track 30.6 -> 29.2 mm
- net /M_SCL: track 109.7 -> 110.4 mm
