File: Schematics & PCB/sensOrb/salp_board_round.kicad_pcb (KiCad board)
At the start: 4 copper layers, 56.2 x 56.2 mm, 63 parts, among them J3 ATTINY3226, J4 POWER, J5 ATTINY3226, J7 READ/WRITE, J8 READ/WRITE, Q1 IRLML6402, Q2 IRLML6402, U1 PN5321A3HN/C106_55, U2 ATtiny3226-S, U3 TP4057, U4 LD1117S33TR, U5 DW01A, Y1 27.12 MHz

Commit message: Silkscreen Fixes
Parts:
- moved BT1 0.10 mm to (157.1, 90.0)
Other:
- board text added: "SALP_Dev_Board V2.0 Initial Design by Owen Pyle Revisions by Jack Cunningham"
Changed lines of the file:
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@@
 		(tags "Through hole pin header THT 1x06 2.54mm single row")
 		(property "Reference" "J6"
-			(at 1 -2.38 0)
+			(at -2.8 -0.78 0)
 			(layer "F.SilkS")
 			(effects
@@
 		(tags "capacitor handsolder")
 		(property "Reference" "C14"
-			(at 0.1 -1.6 90)
+			(at 0.4 -1.7 90)
 			(layer "F.SilkS")
 			(effects
 				(font
-					(size 0.9 0.9)
-					(thickness 0.15)
+					(size 1 0.9)
+					(thickness 0.153)
+					(bold yes)
 				)
 			)
@@
 			(effects
 				(font
-					(size 0.701366 0.701366)
-					(thickness 0.15)
+					(size 1 0.701366)
+					(thickness 0.153)
+					(bold yes)
 				)
 			)
@@
 		(tags "resistor handsolder")
 		(property "Reference" "R11"
-			(at -2.6 0 180)
+			(at -2.6 0.1 180)
 			(layer "F.SilkS")
 			(effects
@@
 				(font
 					(size 1 1)
-					(thickness 0.15)
+					(thickness 0.153)
 				)
 			)
@@
 		(tags "CMS SOT")
 		(property "Reference" "U4"
-			(at -1.2 -4.1 360)
+			(at -1.3 -4.4 360)
 			(layer "F.SilkS")
 			(effects
@@
 		(tags "Through hole pin header THT 1x03 2.54mm single row")
 		(property "Reference" "SEL1"
-			(at 2.7 -2.5 0)
+			(at 2.7 -2.4 0)
 			(layer "F.SilkS")
 			(effects
 				(font
 					(size 1 1)
-					(thickness 0.15)
+					(thickness 0.153)
 				)
 			)
@@
 	(footprint "Battery:BatteryHolder_Keystone_1060_1x2032"
 		(layer "B.Cu")
-		(at 157.1 90.05 90)
+		(at 157.1 89.95 90)
 		(descr "http://www.keyelco.com/product-pdf.cfm?p=726")
 		(tags "CR2032 BR2032 BatteryHolder Battery")
@@
 		(layer "Edge.Cuts")
 	)
-	(gr_text "Bottom-1\nTop-0\n\n00 - HSU/USART\n01 - SPI\n10 - I2C"
-		(at 168.8 70.7 0)
+	(gr_text "SALP_Dev_Board V2.0\nInitial Design by Owen Pyle\nRevisions by Jack Cunningham\n"
+		(at 192.4 87.5 0)
+		(layer "B.SilkS")
+		(effects
+			(font
+				(size 1 0.9)
+				(thickness 0.153)
+				(bold yes)
+			)
+			(justify left bottom mirror)
+		)
+	)
+	(gr_text "Bottom-1\nTop-0\n00 - HSU/USART\n01 - SPI\n10 - I2C"
+		(at 168.4 72.3 0)
 		(layer "F.SilkS")
 		(effects
 			(font
-				(size 0.7 0.7)
-				(thickness 0.15)
+				(size 1 0.7)
+				(thickness 0.153)
 				(bold yes)
 			)
@@
 	)
 	(gr_text "LEFTx2: READ\nRIGHTx2: PROGRAM"
-		(at 173.9 72.6 0)
+		(at 173.4 72.5 0)
 		(layer "F.SilkS")
 		(effects
 			(font
-				(size 0.7 0.7)
-				(thickness 0.1)
+				(size 1 0.7)
+				(thickness 0.153)
+				(bold yes)
 			)
 			(justify left bottom)
@@
 	)
 	(segment
+		(start 157.1 75.3)
+		(end 157.1 72.9)
+		(width 1)
+		(layer "B.Cu")
+		(net 1)
+	)
+	(segment
 		(start 160.2 107.1)
 		(end 160.3 107.2)
@@
 	)
 	(segment
-		(start 157.1 75.4)
-		(end 157.1 72.9)
-		(width 1)
-		(layer "B.Cu")
-		(net 1)
-	)
-	(segment
 		(start 178 109.098223)
 		(end 181.098223 109.098223)
@@
 	)
 	(segment
-		(start 158.2 104.7)
-		(end 160.1 102.8)
+		(start 168.1 101.7)
+		(end 168.1 98.7)
 		(width 0.5)
 		(layer "B.Cu")
@@
 	)
 	(segment
-		(start 168.1 101.7)
-		(end 168.1 98.7)
-		(width 0.5)
+		(start 157.1 104.7)
+		(end 156.1 105.7)
+		(width 1)
+		(layer "B.Cu")
+		(net 2)
+	)
+	(segment
+		(start 158.2 104.7)
+		(end 157.1 104.7)
+		(width 1)
 		(layer "B.Cu")
 		(net 2)
@@
 	)
 	(segment
-		(start 157.1 104.7)
-		(end 158.2 104.7)
-		(width 1)
+		(start 158.2 104.7)
+		(end 160.1 102.8)
+		(width 0.5)
 		(layer "B.Cu")
 		(net 2)
@@
 	)
 	(segment
-		(start 153.7 105.7)
-		(end 156.1 105.7)
-		(width 1)
-		(layer "B.Cu")
-		(net 2)
-	)
-	(segment
 		(start 156.1 105.7)
-		(end 157.1 104.7)
+		(end 153.7 105.7)
 		(width 1)
 		(layer "B.Cu")

Commit message: Silkscreen Fixes
Parts:
- moved D2 0.99 mm to (186.2, 71.5)
Routing:
- net Net-(D2-K): track 4.94 -> 4.15 mm
Changed lines of the file:
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@@
 		(tags "Through hole pin header THT 1x03 2.54mm single row")
 		(property "Reference" "SEL0"
-			(at 1.5 -2.475 0)
+			(at 0.1 -2.475 0)
 			(layer "F.SilkS")
 			(effects
@@
 	(footprint "Diode_SMD:D_1206_3216Metric_Pad1.42x1.75mm_HandSolder"
 		(layer "F.Cu")
-		(at 185.8 70.6 180)
+		(at 186.2125 71.5 180)
 		(descr "Diode SMD 1206 (3216 Metric), square (rectangular) end terminal, IPC_7351 nominal, (Body size source: http://www.tortai-tech.com/upload/download/2011102023233369053.pdf), generated with kicad-footprint-generator")
 		(tags "diode handsolder")
@@
 	)
 	(gr_text "SALP_Dev_Board V2.0\nInitial Design by Owen Pyle\nRevisions by Jack Cunningham\n"
-		(at 192.4 87.5 0)
+		(at 192.5 92 0)
 		(layer "B.SilkS")
 		(effects
@@
 	)
 	(gr_text "Bottom-1\nTop-0\n00 - HSU/USART\n01 - SPI\n10 - I2C"
-		(at 168.4 72.3 0)
+		(at 168.3 72.1 0)
 		(layer "F.SilkS")
 		(effects
@@
 	)
 	(gr_text "LEFTx2: READ\nRIGHTx2: PROGRAM"
-		(at 173.4 72.5 0)
+		(at 173.7 72.5 0)
 		(layer "F.SilkS")
 		(effects
@@
 	)
 	(segment
-		(start 184.46 96.6)
-		(end 185.76 97.9)
+		(start 179.94 74.06)
+		(end 182.5 71.5)
 		(width 0.3)
 		(layer "F.Cu")
@@
 	)
 	(segment
-		(start 183.94 70.6)
-		(end 184.3125 70.6)
-		(width 0.2)
-		(layer "F.Cu")
-		(net 9)
-	)
-	(segment
-		(start 179.94 74.6)
-		(end 183.94 70.6)
+		(start 184.46 96.6)
+		(end 185.76 97.9)
 		(width 0.3)
 		(layer "F.Cu")
@@
 	)
 	(segment
+		(start 184.725 71.5)
+		(end 184.725 71.385)
+		(width 0.3)
+		(layer "F.Cu")
+		(net 9)
+	)
+	(segment
 		(start 181.235 94.435)
 		(end 183.4 96.6)
@@
 	)
 	(segment
+		(start 179.94 74.6)
+		(end 179.94 74.06)
+		(width 0.3)
+		(layer "F.Cu")
+		(net 9)
+	)
+	(segment
+		(start 182.5 71.5)
+		(end 184.725 71.5)
+		(width 0.3)
+		(layer "F.Cu")
+		(net 9)
+	)
+	(segment
 		(start 183.4 96.6)
 		(end 184.46 96.6)
@@
 	)
 	(segment
+		(start 189.555 74.6)
+		(end 189.555 72.8675)
+		(width 0.3)
+		(layer "F.Cu")
+		(net 10)
+	)
+	(segment
 		(start 189.555 72.8675)
-		(end 187.2875 70.6)
+		(end 188.1875 71.5)
 		(width 0.3)
 		(layer "F.Cu")
@@
 	)
 	(segment
-		(start 189.555 74.6)
-		(end 189.555 72.8675)
+		(start 188.1875 71.5)
+		(end 187.7 71.5)
 		(width 0.3)
 		(layer "F.Cu")

Commit message: Silkscreen Fixes
Parts:
- moved J6 0.30 mm to (168.0, 74.8)
- moved BT1 0.10 mm to (157.0, 90.0)
Routing:
- net /M_SCL: track 110.4 -> 111.8 mm
- net /PA7: track 30.7 -> 31.8 mm
Other:
- board text added: "SALP_Dev_Board V2.0 Initial Design by Owen Pyle Revisions by Jack Cunningham 7/7/25"
- board text removed: "SALP_Dev_Board V2.0 Initial Design by Owen Pyle Revisions by Jack Cunningham"

Commit message: Placement/Clearance FIxes
Parts:
- moved C21 0.80 mm to (145.0, 98.4)
- moved U5 0.59 mm to (148.3, 103.2)
- moved BT1 0.51 mm to (156.5, 89.8)
- moved J6 0.50 mm to (167.5, 74.9)
- moved R7 0.50 mm to (152.2, 105.7)
- moved R8 0.50 mm to (147.0, 99.2)
- moved C11 0.34 mm to (163.7, 77.9)
- moved Antenna 0.30 mm to (146.2, 80.5)
- moved J3 0.30 mm to (192.9, 81.1)
Routing:
- net /M_SCL: track 111.8 -> 110.1 mm
- net Net-(J6-Pin_2): track 10.4 -> 11.5 mm
- net GND: track 102.5 -> 101.8 mm
- net Net-(U5-CS): track 4.48 -> 5.11 mm
- net +BAT: track 30.5 -> 31.1 mm
