File: Schematics & PCB/sensOrb/salp_board_round.kicad_pcb (KiCad board)
At the start: 4 copper layers, 56.2 x 56.2 mm, 63 parts, among them J3 ATTINY3226, J4 POWER, J5 ATTINY3226, J7 READ/WRITE, J8 READ/WRITE, Q1 IRLML6402, Q2 IRLML6402, U1 PN5321A3HN/C106_55, U2 ATtiny3226-S, U3 TP4057, U4 LD1117S33TR, U5 DW01A, Y1 27.12 MHz

Commit message: Fixes
Parts:
- renumbered Antenna to J1, SEL0 to J10, SEL1 to J9
Connections:
- C12 pad 2: Net-(J1-Pin_2) -> GND
- C13 pad 1: Net-(J1-Pin_2) -> GND
- C5 pad 2: Net-(J1-Pin_2) -> GND
- C6 pad 1: Net-(J1-Pin_2) -> GND
- J1 pad 2: Net-(J1-Pin_2) -> GND
- L1 pad 2: /TX1 -> /TX2
- L2 pad 2: /TX2 -> /TX1
Routing:
- net GND: track 100.6 -> 127.0 mm
- net Net-(J1-Pin_2): track 26.4 -> 0.00 mm
- net /TX2: track 16.8 -> 21.6 mm
- net /TX1: track 21.3 -> 19.7 mm
- net /AVDD: track 40.8 -> 40.7 mm, vias 2 -> 0

Commit message: Fixes To Battery Management
Parts:
- Q1, Q2: value IRLML6402 -> DMN10H220L
- moved Q2 7.67 mm to (153.6, 108.9), turned to -90 degrees
- moved Q1 6.67 mm to (159.6, 110.4), turned to -90 degrees
- moved C23 5.32 mm to (158.0, 107.4)
- moved R8 0.10 mm to (147.0, 99.1)
Connections:
- Q1 pad 3: +BAT -> Net-(Q1-D)
- Q2 pad 3: +3.3V -> Net-(Q1-D)
Routing:
- net Net-(Q2-G): track 18.9 -> 9.13 mm, vias 2 -> 0
- net +BAT: track 31.1 -> 24.2 mm, vias 5 -> 3
- net Net-(Q1-G): track 7.54 -> 14.2 mm, vias 0 -> 2
- net Net-(Q1-D): track 0.00 -> 6.60 mm
- net +3.3V: track 36.6 -> 34.0 mm, vias 6 -> 5
- net GND: track 127.0 -> 128.5 mm, vias 20 -> 19
Other:
- board text added: "SALP_Dev_Board V2.0 Initial Design by Owen Pyle Revisions by Jack Cunningham 7/10/25"
- board text removed: "SALP_Dev_Board V2.0 Initial Design by Owen Pyle Revisions by Jack Cunningham 7/7/25"
