File: Schematics & PCB/sensOrb_JackRev_STM32/PN7160_STM32.kicad_pcb (KiCad board)
At the start: 2 copper layers, 0 parts

Commit message: PCB Changes
Parts:
- added C1: 2.2u, Capacitor_SMD:C_0805_2012Metric_Pad1.18x1.45mm_HandSolder, F.Cu at (168.5, 91.0)
- added C10: 1u, Capacitor_SMD:C_0805_2012Metric_Pad1.18x1.45mm_HandSolder, F.Cu at (157.3, 104.7)
- added C11: 0.1u, Capacitor_SMD:C_0805_2012Metric_Pad1.18x1.45mm_HandSolder, F.Cu at (154.4, 111.5)
- added C12: 0.1u, Capacitor_SMD:C_0805_2012Metric_Pad1.18x1.45mm_HandSolder, F.Cu at (171.2, 114.3)
- added C13: 1u, Capacitor_SMD:C_0805_2012Metric_Pad1.18x1.45mm_HandSolder, F.Cu at (138.7, 78.0)
- added C14: 1u, Capacitor_SMD:C_0805_2012Metric_Pad1.18x1.45mm_HandSolder, F.Cu at (142.6, 83.4)
- added C15: 10u, Capacitor_SMD:C_0805_2012Metric_Pad1.18x1.45mm_HandSolder, F.Cu at (151.1, 86.6)
- added C16: 10u, Capacitor_SMD:C_0805_2012Metric_Pad1.18x1.45mm_HandSolder, F.Cu at (152.5, 90.4)
- added C17: 10nF, Capacitor_SMD:C_0805_2012Metric_Pad1.18x1.45mm_HandSolder, B.Cu at (142.7, 95.4)
- added C18: 100nF, Capacitor_SMD:C_0805_2012Metric_Pad1.18x1.45mm_HandSolder, B.Cu at (146.6, 95.4)
- added C19: 0.1u, Capacitor_SMD:C_0805_2012Metric_Pad1.18x1.45mm_HandSolder, B.Cu at (160.2, 104.0)
- added C2: 1.5p, Capacitor_SMD:C_0805_2012Metric_Pad1.18x1.45mm_HandSolder, F.Cu at (160.0, 102.5)
- added C20: 2.2u, Capacitor_SMD:C_0805_2012Metric_Pad1.18x1.45mm_HandSolder, B.Cu at (168.5, 105.5)
- added C21: 2.2u, Capacitor_SMD:C_0805_2012Metric_Pad1.18x1.45mm_HandSolder, B.Cu at (166.5, 105.5)
- added C22: 2.2u, Capacitor_SMD:C_0805_2012Metric_Pad1.18x1.45mm_HandSolder, B.Cu at (156.7, 96.8)
- added C23: 2.2u, Capacitor_SMD:C_0805_2012Metric_Pad1.18x1.45mm_HandSolder, B.Cu at (155.0, 94.7)
- added C24: 4.7u, Capacitor_SMD:C_0805_2012Metric_Pad1.18x1.45mm_HandSolder, B.Cu at (153.5, 100.3)
- added C25: 0.1u, Capacitor_SMD:C_0805_2012Metric_Pad1.18x1.45mm_HandSolder, B.Cu at (153.5, 103.5)
- added C26: 1u, Capacitor_SMD:C_0805_2012Metric_Pad1.18x1.45mm_HandSolder, B.Cu at (176.5, 103.0)
- added C27: 4.7u, Capacitor_SMD:C_0805_2012Metric_Pad1.18x1.45mm_HandSolder, B.Cu at (168.0, 101.6)
- added C28: 10p, Capacitor_SMD:C_0805_2012Metric_Pad1.18x1.45mm_HandSolder, B.Cu at (152.5, 90.0)
- added C29: 10p, Capacitor_SMD:C_0805_2012Metric_Pad1.18x1.45mm_HandSolder, B.Cu at (157.5, 90.0)
- added C3: 1.5p, Capacitor_SMD:C_0805_2012Metric_Pad1.18x1.45mm_HandSolder, F.Cu at (160.5, 111.1)
- added C30: 1n, Capacitor_SMD:C_0603_1608Metric_Pad1.08x0.95mm_HandSolder, B.Cu at (164.0, 103.6)
- added C31: 1n, Capacitor_SMD:C_0603_1608Metric_Pad1.08x0.95mm_HandSolder, B.Cu at (162.5, 103.6)
- added C32: 330p, Capacitor_SMD:C_0603_1608Metric_Pad1.08x0.95mm_HandSolder, B.Cu at (154.1, 111.0)
- added C33: 330p, Capacitor_SMD:C_0603_1608Metric_Pad1.08x0.95mm_HandSolder, B.Cu at (158.0, 111.0)
- added C34: 82p, Capacitor_SMD:C_0201_0603Metric_Pad0.64x0.40mm_HandSolder, B.Cu at (153.5, 113.0)
- added C35: 82p, Capacitor_SMD:C_0201_0603Metric_Pad0.64x0.40mm_HandSolder, B.Cu at (159.0, 113.0)
- added C36: 150p, Capacitor_SMD:C_0603_1608Metric_Pad1.08x0.95mm_HandSolder, B.Cu at (154.5, 116.0)
- added C37: 150p, Capacitor_SMD:C_0603_1608Metric_Pad1.08x0.95mm_HandSolder, B.Cu at (158.0, 116.0)
- added C4: 10p, Capacitor_SMD:C_0805_2012Metric_Pad1.18x1.45mm_HandSolder, F.Cu at (159.5, 117.5)
- added C5: 10p, Capacitor_SMD:C_0805_2012Metric_Pad1.18x1.45mm_HandSolder, F.Cu at (163.8, 111.4)
- added C6: 0.1u, Capacitor_SMD:C_0805_2012Metric_Pad1.18x1.45mm_HandSolder, F.Cu at (157.3, 112.7)
- added C7: 0.1u, Capacitor_SMD:C_0805_2012Metric_Pad1.18x1.45mm_HandSolder, F.Cu at (157.3, 110.7)
- added C8: 0.1u, Capacitor_SMD:C_0805_2012Metric_Pad1.18x1.45mm_HandSolder, F.Cu at (157.3, 108.7)
- added C9: 0.1u, Capacitor_SMD:C_0805_2012Metric_Pad1.18x1.45mm_HandSolder, F.Cu at (157.3, 106.7)
- added D1: RED LED, LED_SMD:LED_0603_1608Metric_Pad1.05x0.95mm_HandSolder, F.Cu at (138.7, 75.9)
- added D2: BLUE LED, LED_SMD:LED_0603_1608Metric_Pad1.05x0.95mm_HandSolder, F.Cu at (164.3, 86.7)
- added D3: GREEN LED, LED_SMD:LED_0603_1608Metric_Pad1.05x0.95mm_HandSolder, F.Cu at (161.3, 86.8)
- added D5: BAT54CW, Package_TO_SOT_SMD:SOT-323_SC-70, F.Cu at (149.0, 84.4)
- added H1: MountingHole_Pad, MountingHole:MountingHole_2.2mm_M2_Pad, F.Cu at (168.0, 118.0)
- added H2: MountingHole_Pad, MountingHole:MountingHole_2.2mm_M2_Pad, F.Cu at (132.0, 82.0)
- added J1: USB4215-03-A_REVA, footprints:GCT_USB4215-03-A_REVA, F.Cu at (150.0, 75.0)
- added J10: Conn_01x02, Connector_JST:JST_XH_B2B-XH-A_1x02_P2.50mm_Vertical, F.Cu at (158.4, 78.0)
- added J11: STM32 Optional I/O, Connector_PinSocket_2.54mm:PinSocket_2x09_P2.54mm_Vertical, F.Cu at (171.4, 110.4)
- added J12: Antenna_Conn, Connector_JST:JST_ACH_BM02B-ACHSS-GAN-ETF_1x02-1MP_P1.20mm_Vertical, B.Cu at (156.6, 123.6)
- added J2: Conn_01x04, Connector_JST:JST_XH_B4B-XH-A_1x04_P2.50mm_Vertical, B.Cu at (146.3, 120.8)
- added J3: Conn_01x04, Connector_JST:JST_XH_B4B-XH-A_1x04_P2.50mm_Vertical, B.Cu at (141.8, 114.1)
- added J4: Conn_01x04, Connector_JST:JST_XH_B4B-XH-A_1x04_P2.50mm_Vertical, B.Cu at (141.8, 107.3)
- added J5: Conn_01x04, Connector_JST:JST_XH_B4B-XH-A_1x04_P2.50mm_Vertical, B.Cu at (133.7, 97.5)
- added J6: Conn_01x04, Connector_JST:JST_XH_B4B-XH-A_1x04_P2.50mm_Vertical, B.Cu at (127.2, 91.8)
- added J7: Conn_01x04, Connector_JST:JST_XH_B4B-XH-A_1x04_P2.50mm_Vertical, B.Cu at (140.6, 91.5)
- added J8: IMU Top, Connector_PinSocket_2.54mm:PinSocket_1x06_P2.54mm_Vertical, F.Cu at (129.1, 102.5)
- added J9: IMU Bottom, Connector_PinSocket_2.54mm:PinSocket_1x06_P2.54mm_Vertical, F.Cu at (147.0, 102.5)
- added L1: 4.7u, 500mA, Inductor_SMD:L_0805_2012Metric_Pad1.05x1.20mm_HandSolder, F.Cu at (155.1, 91.5)
- added L2: 160n, Inductor_SMD:L_0603_1608Metric_Pad1.05x0.95mm_HandSolder, B.Cu at (158.5, 106.0)
- added L3: 160n, Inductor_SMD:L_0603_1608Metric_Pad1.05x0.95mm_HandSolder, B.Cu at (155.0, 106.0)
- added R1: 5.1K, Resistor_SMD:R_0805_2012Metric_Pad1.20x1.40mm_HandSolder, F.Cu at (152.5, 81.6)
- added R10: 200k, Resistor_SMD:R_0805_2012Metric_Pad1.20x1.40mm_HandSolder, F.Cu at (158.0, 90.4)
- added R11: 100, Resistor_SMD:R_0603_1608Metric_Pad0.98x0.95mm_HandSolder, F.Cu at (164.3, 90.1)
- added R12: 220, Resistor_SMD:R_0603_1608Metric_Pad0.98x0.95mm_HandSolder, F.Cu at (161.3, 90.2)
- added R13: 10k, Resistor_SMD:R_0805_2012Metric_Pad1.20x1.40mm_HandSolder, B.Cu at (134.0, 103.1)
- added R14: 10k, Resistor_SMD:R_0805_2012Metric_Pad1.20x1.40mm_HandSolder, B.Cu at (168.5, 94.0)
- added R15: 10k, Resistor_SMD:R_0805_2012Metric_Pad1.20x1.40mm_HandSolder, B.Cu at (166.5, 89.5)
- added R16: 10k, Resistor_SMD:R_0805_2012Metric_Pad1.20x1.40mm_HandSolder, B.Cu at (168.5, 90.0)
- added R19: 2.2k, Resistor_SMD:R_0805_2012Metric_Pad1.20x1.40mm_HandSolder, B.Cu at (155.5, 108.5)
- added R2: 5.1K, Resistor_SMD:R_0805_2012Metric_Pad1.20x1.40mm_HandSolder, F.Cu at (146.8, 81.6)
- added R20: 1.54, Resistor_SMD:R_0603_1608Metric_Pad0.98x0.95mm_HandSolder, B.Cu at (153.5, 119.0)
- added R21: 1.54, Resistor_SMD:R_0603_1608Metric_Pad0.98x0.95mm_HandSolder, B.Cu at (159.0, 119.0)
- added R22: 2.2k, Resistor_SMD:R_0805_2012Metric_Pad1.20x1.40mm_HandSolder, B.Cu at (159.5, 109.0)
- added R3: 4.7k, Resistor_SMD:R_0805_2012Metric_Pad1.20x1.40mm_HandSolder, F.Cu at (147.0, 98.5)
- added R4: 4.7k, Resistor_SMD:R_0805_2012Metric_Pad1.20x1.40mm_HandSolder, F.Cu at (150.0, 97.0)
- added R5: 10k, Resistor_SMD:R_0805_2012Metric_Pad1.20x1.40mm_HandSolder, F.Cu at (152.3, 111.5)
- added R7: 10k, Resistor_SMD:R_0805_2012Metric_Pad1.20x1.40mm_HandSolder, F.Cu at (168.5, 95.0)
- added R8: 5.1K, Resistor_SMD:R_0805_2012Metric_Pad1.20x1.40mm_HandSolder, F.Cu at (142.5, 76.4)
- added R9: 1.8M, Resistor_SMD:R_0805_2012Metric_Pad1.20x1.40mm_HandSolder, F.Cu at (158.2, 86.5)
- added SW1: SW_SPST, Button_Switch_SMD:SW_Tactile_SPST_NO_Straight_CK_PTS636Sx25SMTRLFS, F.Cu at (153.2, 104.5)
- added SW2: SW_SPST, Button_Switch_SMD:SW_Tactile_SPST_NO_Straight_CK_PTS636Sx25SMTRLFS, F.Cu at (167.0, 110.1)
- added U1: PN7160A1HN/C100E, footprints:QFN40_PN7160_NXP-M, B.Cu at (162.7, 97.0)
- added U3: STM32F411CEU6, footprints:QFN50P700X700X60-49N, F.Cu at (163.1, 96.8)
- added U4: TLV75533PDBVR, footprints:DBV0005A_L, F.Cu at (142.6, 79.8)
- added U5: TPS61070DDCR, footprints:DDC0006A_L, F.Cu at (155.3, 86.5)
- added U6: TCA9548APWR, Package_SO:TSSOP-24_4.4x7.8mm_P0.65mm, B.Cu at (141.2, 100.3)
- added XTAL1: XRCGB27M120F3M00R0, footprints:XTAL_XRCGB27M120F3M00R0_MUR, B.Cu at (155.0, 91.5)
- added Y1: ABS07-32.768KHZ-T, footprints:XTAL_ABS07-32.768KHZ-T, F.Cu at (160.5, 107.0)
- added Y2: TSX-3225_24.0000MF20G-AC3, footprints:XTAL_TSX-3225_24.0000MF20G-AC3, F.Cu at (163.3, 115.3)
Routing:
- net GND: track 0.00 -> 228.0 mm, vias 0 -> 25
- net +3.3V: track 0.00 -> 142.6 mm, vias 0 -> 12
- net /SCL: track 0.00 -> 84.9 mm, vias 0 -> 5
- net /SDA: track 0.00 -> 74.4 mm, vias 0 -> 3
- net /IMU_RST: track 0.00 -> 43.7 mm, vias 0 -> 2
- net +5V: track 0.00 -> 40.8 mm
- net /IMU_INT: track 0.00 -> 38.2 mm
- net /PA12: track 0.00 -> 28.3 mm, vias 0 -> 2
- net /TVDD: track 0.00 -> 27.9 mm, vias 0 -> 6
- net /PA11: track 0.00 -> 26.6 mm, vias 0 -> 2
- net Net-(SW1-A): track 0.00 -> 22.2 mm, vias 0 -> 2
- net /BAT_IN: track 0.00 -> 22.2 mm, vias 0 -> 1
- net Net-(U3-PH0-OSC_IN): track 0.00 -> 20.0 mm
- net /SC0: track 0.00 -> 19.7 mm
- net /SD0: track 0.00 -> 18.8 mm
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- added copper zone on In2.Cu, net +3.3V
- added copper zone on In1.Cu, net GND
Other:
- board outline added: 56.2 x 56.2 mm
- copper layers 2 -> 4
- board text added: "BOOT->"
- board text added: "RESET->"
