File: Schematics & PCB/sensOrb_JackRev_STM32/PN7160_STM32.kicad_pcb (KiCad board)
At the start: 4 copper layers, 59.4 x 59.4 mm, 87 parts, among them J1 USB4215-03-A_REVA, J10 Conn_01x02, J11 STM32 Optional I/O, J12 Antenna_Conn, J2 Conn_01x04, J3 Conn_01x04, J4 Conn_01x04, J5 Conn_01x04, J6 Conn_01x04, J7 Conn_01x04, J8 IMU Top, J9 IMU Bottom, SW1 SW_SPST, SW2 SW_SPST, U1 PN7160A1HN/C100E, U3 STM32F411CEU6, U4 TLV75533PDBVR, U5 TPS61070DDCR, U6 TCA9548APWR, Y1 ABS07-32.768KHZ-T, Y2 TSX-3225_24.0000MF20G-AC3

Commit message: Fixes to some footprints
Parts:
- C2, C28, C29, C3, C4, C5: footprint Capacitor_SMD:C_0805_2012Metric_Pad1.18x1.45mm_HandSolder -> Capacitor_SMD:C_0402_1005Metric_Pad0.74x0.62mm_HandSolder
- moved C28 1.77 mm to (167.0, 85.4), turned to 90 degrees
Routing:
- net GND: track 186.5 -> 188.6 mm
- net /XTAL2: track 14.0 -> 12.6 mm
