File: Schematics & PCB/sensOrb_JackRev_STM32/PN7160_STM32.kicad_sch (KiCad schematic)
At the start: 87 parts, among them J1 USB4215-03-A_REVA, J10 Conn_01x02, J11 STM32 Optional I/O, J12 Antenna_Conn, J2 Conn_01x04, J3 Conn_01x04, J4 Conn_01x04, J5 Conn_01x04, J6 Conn_01x04, J7 Conn_01x04, J8 IMU Top, J9 IMU Bottom, SW1 D6R90F2LFS, SW2 D6R90F2LFS, U1 PN7160A1HN/C100E, U3 STM32F411CEU6, U4 TLV75533PDBVR, U5 TPS61070DDCR, U6 TCA9548APWR, Y1 ABS07-32.768KHZ-T, Y2 TSX-3225_24.0000MF20G-AC3

Commit message: PCB Changes
Parts:
- removed SW1, SW2: D6R90F2LFS, footprints:D6R90_CNK, symbol SPST-NO_D6R90F2LFS:D6R90F2LFS
- added SW1, SW2: SW_SPST, Button_Switch_SMD:SW_Tactile_SPST_NO_Straight_CK_PTS636Sx25SMTRLFS, symbol Switch:SW_SPST
- J2, J3, J4, J5, J6, J7: footprint Connector_JST:JST_XH_B4B-XH-AM_1x04_P2.50mm_Vertical -> Connector_JST:JST_XH_B4B-XH-A_1x04_P2.50mm_Vertical
- R19: footprint Resistor_SMD:R_0815_2038Metric_Pad1.20x4.05mm_HandSolder -> Resistor_SMD:R_0805_2012Metric_Pad1.20x1.40mm_HandSolder
Connections:
- net +3.3V: now also SW1.2 (B); no longer J8.1 (Pin_1)
- net +5V: now also J11.18 (Pin_18); no longer J11.9 (Pin_9)
- net GND: now also J11.16 (Pin_16), SW2.1 (A); no longer J11.10 (Pin_10)
- net PA1: now also J11.3 (Pin_3); no longer J11.2 (Pin_2)
- net PA2: now also J11.5 (Pin_5); no longer J11.3 (Pin_3)
- net PA3: now also J11.7 (Pin_7); no longer J11.4 (Pin_4)
- net PA6: now also J11.9 (Pin_9); no longer J11.5 (Pin_5)
- net PA7: now also J11.11 (Pin_11); no longer J11.6 (Pin_6)
- net PA8: now also J11.6 (Pin_6); no longer J11.7 (Pin_7)
- net PB1: now also J11.13 (Pin_13); no longer J11.11 (Pin_11)
- net PB12: now also J11.17 (Pin_17); no longer J11.16 (Pin_16)
- net PB13: now also J11.2 (Pin_2); no longer J11.17 (Pin_17)
- net PB14: now also J11.4 (Pin_4); no longer J11.18 (Pin_18)
- net PB3: now also J11.10 (Pin_10); no longer J11.12 (Pin_12)
- net PB4: now also J11.12 (Pin_12); no longer J11.13 (Pin_13)
- net at C11.1, R5.2, U3.44 (BOOT0): now also SW1.1 (A)
- net at C12.1, U3.7 (NRST): now also SW2.2 (B)
- new net BT: J8.1 (Pin_1)
- no-connect marks 25 -> 26
Other:
- moved on the sheet: C12
