File: Schematics & PCB/sensOrb_JackRev_STM32/PN7160_STM32.kicad_sch (KiCad schematic)
At the start: 87 parts, among them J1 USB4215-03-A_REVA, J10 Conn_01x02, J11 STM32 Optional I/O, J12 Antenna_Conn, J2 Conn_01x04, J3 Conn_01x04, J4 Conn_01x04, J5 Conn_01x04, J6 Conn_01x04, J7 Conn_01x04, J8 IMU Top, J9 IMU Bottom, SW1 SW_SPST, SW2 SW_SPST, U1 PN7160A1HN/C100E, U3 STM32F411CEU6, U4 TLV75533PDBVR, U5 TPS61070DDCR, U6 TCA9548APWR, Y1 ABS07-32.768KHZ-T, Y2 TSX-3225_24.0000MF20G-AC3

Commit message: Finalized PCB Layout
Connections:
- net +3.3V: now also J11.18 (Pin_18)
- net +5V: no longer J11.18 (Pin_18)
Changed lines of the file:
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@@
 	)
 	(junction
+		(at 29.21 97.79)
+		(diameter 0)
+		(color 0 0 0 0)
+	)
+	(junction
 		(at 191.77 118.11)
 		(diameter 0)
@@
 	)
 	(junction
-		(at 29.21 97.79)
-		(diameter 0)
-		(color 0 0 0 0)
-	)
-	(junction
 		(at 161.29 31.75)
 		(diameter 0)
@@
 		)
 	)
+	(wire
+		(pts
+			(xy 29.21 97.79) (xy 34.29 97.79)
+		)
+		(stroke
+			(width 0)
+			(type default)
+		)
+	)
 	(polyline
 		(pts
@@
 	(wire
 		(pts
-			(xy 34.29 97.79) (xy 29.21 97.79)
-		)
-		(stroke
-			(width 0)
-			(type default)
-		)
-	)
-	(wire
-		(pts
 			(xy 39.37 106.68) (xy 50.8 106.68)
 		)
@@
 			)
 		)
-		(property "Value" "+5V"
+		(property "Value" "+3.3V"
 			(at 279.654 121.158 90)
 			(effects

Commit message: Code file moves+PCB pngs
Other:
- title: STM32-PN7160 SALP Integration -> STM32-PN7160 Integration
- moved on the sheet: C30, C31, C32, C33, C34, C35, C36, C37, L2, L3, R19, R20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
