File: Schematics & PCB/sensOrb_Baro_Unit/sensOrb_Baro_Unit.kicad_pcb (KiCad board)
At the start: 2 copper layers, 25.5 x 17 mm, 7 parts, among them J11 Conn_01x04, U1 MS583730BA01-50

Commit message: Fixes to some footprints
Parts:
- J11: footprint Connector_JST:JST_XH_B4B-XH-AM_1x04_P2.50mm_Vertical -> Connector_JST:JST_XH_B4B-XH-A_1x04_P2.50mm_Vertical
Changed lines of the file:
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@@
 		(embedded_fonts no)
 	)
-	(footprint "Connector_JST:JST_XH_B4B-XH-AM_1x04_P2.50mm_Vertical"
+	(footprint "Connector_JST:JST_XH_B4B-XH-A_1x04_P2.50mm_Vertical"
 		(layer "B.Cu")
 		(at 143.5 99.5)
-		(descr "JST XH series connector, B4B-XH-AM, with boss (http://www.jst-mfg.com/product/pdf/eng/eXH.pdf), generated with kicad-footprint-generator")
-		(tags "connector JST XH vertical boss")
+		(descr "JST XH series connector, B4B-XH-A (http://www.jst-mfg.com/product/pdf/eng/eXH.pdf), generated with kicad-footprint-generator")
+		(tags "connector JST XH vertical")
 		(property "Reference" "J11"
-			(at 12 -2.5 180)
+			(at 12 -3 180)
 			(layer "B.SilkS")
 			(effects
@@
 			)
 		)
-		(property "Datasheet" "~"
+		(property "Datasheet" ""
 			(at 0 0 180)
 			(layer "B.Fab")
@@
 			)
 		)
-		(property "Description" "Generic connector, single row, 01x04, script generated (kicad-library-utils/schlib/autogen/connector/)"
+		(property "Description" ""
 			(at 0 0 180)
 			(layer "B.Fab")
@@
 		)
 		(fp_line
+			(start -1.8 -2.75)
+			(end 3.75 -2.75)
+			(stroke
+				(width 0.12)
+				(type solid)
+			)
+			(layer "B.SilkS")
+		)
+		(fp_line
 			(start -1.8 0.2)
-			(end -1.8 -1.14)
+			(end -1.8 -2.75)
 			(stroke
 				(width 0.12)
@@
 		)
 		(fp_line
-			(start 3.75 -2.75)
-			(end -0.74 -2.75)
-			(stroke
-				(width 0.12)
-				(type solid)
-			)
-			(layer "B.SilkS")
-		)
-		(fp_line
 			(start 9.3 -2.75)
 			(end 3.75 -2.75)
@@
 				(justify mirror)
 			)
-		)
-		(pad "" np_thru_hole circle
-			(at -1.6 -2)
-			(size 1.2 1.2)
-			(drill 1.2)
-			(layers "*.Cu" "*.Mask")
 		)
 		(pad "1" thru_hole roundrect
@@
 		)
 		(embedded_fonts no)
-		(model "${KICAD9_3DMODEL_DIR}/Connector_JST.3dshapes/JST_XH_B4B-XH-AM_1x04_P2.50mm_Vertical.step"
+		(model "${KICAD9_3DMODEL_DIR}/Connector_JST.3dshapes/JST_XH_B4B-XH-A_1x04_P2.50mm_Vertical.step"
 			(offset
 				(xyz 0 0 0)

Commit message: Output Files Made
Parts:
- C1, R1, R2: moved to B.Cu
- moved H1 0.50 mm to (138.0, 102.0)
- moved H2 0.50 mm to (156.5, 102.0)
- moved R1 0.50 mm to (141.5, 105.0)
- moved R2 0.50 mm to (141.5, 108.5)
Routing:
- net GND: track 33.3 -> 49.2 mm, vias 1 -> 2
- net +3.3V: track 21.2 -> 22.3 mm, vias 0 -> 2
- net /SD0: track 13.6 -> 14.1 mm, vias 1 -> 2
- net /SC0: track 11.6 -> 12.1 mm, vias 1 -> 2
Other:
- board size 25.5 x 17 mm -> 24.5 x 17 mm
